File: EAGLE/vr98/vr98-revA.brd (EAGLE design)
At the start: 369.5 x 121.8 mm, 433 parts, among them Q1 2N7002, Q2 DMG2305UX-7, Q3 IRLML6401, Q4 2N2222, U1 STM32F411CEU7, U2 74HC589A_DT, U3 74HC589A_DT, U4 74HC589A_DT, U5 M25C, Y1 32.768kHz ±20ppm 6pF, Y2 25MHz 9pF

Commit message: wip
Parts:
- moved J1 122.0 mm to (109.8, 14.3)
- moved U$3 110.1 mm to (362.0, 42.0), turned to 180 degrees
- moved C20 25.1 mm to (98.9, 169.6)
- moved C21 25.1 mm to (95.1, 169.6)
- moved C22 25.1 mm to (91.3, 169.6)
- moved C23 25.1 mm to (87.5, 169.6)
- moved C24 25.1 mm to (83.7, 169.6)
- moved C25 25.1 mm to (79.8, 169.6)
- moved C26 25.1 mm to (76.0, 169.6)
- moved C27 25.1 mm to (72.2, 169.6)
- moved C28 25.1 mm to (68.4, 169.6)
- moved D107 25.1 mm to (64.6, 169.6)
- moved D201 25.1 mm to (58.2, 169.6)
- moved D202 25.1 mm to (51.9, 169.6)
- moved U3 3.54 mm to (164.0, 103.0)
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Connections:
- net COL10: now also U3.4; no longer U3.5
- net COL11: now also D95.C, U3.5; no longer U3.6
- net COL12: now also D96.C, U3.6; no longer D95.C, U4.1
- net COL13: now also D97.C, U3.7; no longer D96.C, U4.2
- net COL14: now also U4.1; no longer D97.C, U4.3
- net COL15: now also U4.2; no longer U4.4
- net COL16: now also U4.3; no longer U4.5
- net COL17: now also U4.4; no longer U4.6
- net COL6: now also U2.7; no longer U3.1
- net COL7: now also U3.1; no longer U3.2
- net COL8: now also U3.2; no longer U3.3
- net COL9: now also U3.3; no longer U3.4
- net GND: now also U4.5, U4.6; no longer U2.7, U3.7

Commit message: wip
Parts:
- removed U$1, U$10, U$11, U$12, U$13, U$14, U$15, U$16, U$17, U$18, U$19, U$2, U$20, U$21, U$22, U$23, U$24, U$25, U$26, U$27, U$6, U$7, U$8, U$9: TEST_PAD, ts_keyboards:TEST_PAD
- turned D1 to 270 degrees
- turned U_LED1 to 180 degrees
- turned U_LED2 to 180 degrees
Connections:
- net COL0: no longer U$11.P$1
- net COL1: no longer U$12.P$1
- net COL10: no longer U$21.P$1
- net COL11: no longer U$22.P$1
- net COL12: no longer U$23.P$1
- net COL13: no longer U$24.P$1
- net COL14: no longer U$25.P$1
- net COL15: no longer U$26.P$1
- net COL16: no longer U$27.P$1
- net COL17: no longer U$1.P$1
- net COL2: no longer U$13.P$1
- net COL3: no longer U$14.P$1
- net COL4: no longer U$15.P$1
- net COL5: no longer U$16.P$1
- net COL6: no longer U$17.P$1
- net COL7: no longer U$18.P$1
- net COL8: no longer U$19.P$1
- net COL9: no longer U$20.P$1
- net ROW0: no longer U$2.P$1
- net ROW1: no longer U$6.P$1
- net ROW2: no longer U$7.P$1
- net ROW3: no longer U$8.P$1
- net ROW4: no longer U$9.P$1
- net ROW5: no longer U$10.P$1

Commit message: wip
Parts:
- removed C31: 100nF, rcl:C0603
- removed Q3: IRLML6401, SparkFun-DiscreteSemi:SOT23-3
- removed Q4: 2N2222, SparkFun-DiscreteSemi:SOT23-3
- removed R72: 1K, rcl:R0603
- removed R73: 100K, rcl:R0603
- added U6: TPS22995H-Q1, __untitled:SOT-23-THIN-6_DDC_TEX
- R71: value 100K -> 1K
- U1: value STM32F411CEU7 -> STM32F411CEU7THERM; device st:UFQFPN-48_7X7X0P55MM -> st:UFQFPN-48_7X7X0P55MM-THERM
- moved RA1 283.3 mm to (342.4, 103.5)
- moved JPWM 277.4 mm to (298.0, 19.0), turned to 180 degrees
- moved C17 274.1 mm to (285.0, 67.0), turned to 90 degrees
- moved C16 265.2 mm to (282.0, 67.0), turned to 90 degrees
- moved C27 262.6 mm to (327.0, 106.0), turned to 180 degrees
- moved JSPI@2 248.0 mm to (259.0, 19.0), turned to 270 degrees
- moved D00 242.6 mm to (284.0, 90.0), turned to 270 degrees
- moved JI2C 240.3 mm to (264.8, 19.1)
- moved C28 240.3 mm to (264.6, 30.7), turned to 90 degrees
- moved R37 239.2 mm to (239.4, 62.0)
- moved R44 234.2 mm to (358.9, 35.3)
- moved R43 234.0 mm to (363.7, 35.3)
- moved C15 233.0 mm to (290.0, 35.6), turned to 270 degrees
- moved C24 225.1 mm to (296.0, 95.0), turned to 270 degrees
- moved C13 220.5 mm to (295.0, 42.8), turned to 270 degrees
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Connections:
- net 5V_SELECT renamed VCC_LED
- net N$122 renamed Y1O
- net N$138 renamed Y2I
- net N$139 renamed Y2O
- net N$143 renamed VREF+
- net N$146 renamed RESET
- net N$79 renamed Y1I
- removed net LED_VCC: C31.1, J_5V.1, Q3.3
- removed net N$147: Q4.3, R72.1
- removed net N$148: C31.2, Q3.1, R71.1, R72.2
- removed net N$153: RA8.4, U_LED1.18
- removed net N$70: Q4.1, R73.1
- removed net UDB_DP: R46.1
- new net LOAD_SWITCH_OUT: J_5V.1, U6.5
- new net N$122: RA8.2, U_LED1.15
- new net N$79: RA8.1, U_LED1.18
- net BLU1: now also RA9.6; no longer RA9.2
- net BLU2: now also RA8.8; no longer RA8.5
- net BLU3: now also RA8.6; no longer RA8.2
- net BLU4: now also RA9.8; no longer RA9.5
- net COL0: now also RA4.8; no longer RA1.8
- net COL1: now also RA4.7; no longer RA1.2
- net COL10: now also RA2.5; no longer RA3.3
- net COL11: now also RA3.8; no longer RA3.5
- net COL12: now also RA3.7; no longer RA4.8
- net COL13: now also RA3.6; no longer RA4.2
- net COL14: now also RA1.8; no longer RA4.3
- net COL15: now also RA1.7; no longer RA4.5
- net COL16: now also RA1.6; no longer RA5.8
- net COL17: now also RA1.5; no longer RA5.2
- net COL2: now also RA4.6; no longer RA1.3
- net COL3: now also RA4.5; no longer RA1.5
- net COL4: now also RA5.8; no longer RA2.8
- net COL5: now also RA5.7; no longer RA2.2
- net COL6: now also RA5.6; no longer RA2.3
- net COL7: now also RA2.8; no longer RA2.5
- net COL8: now also RA2.7; no longer RA3.8
- net COL9: now also RA2.6; no longer RA3.2
- net GND: now also R71.1, U1.49@1, U1.49@10, U1.49@11, U1.49@12, U1.49@13, U1.49@14, U1.49@15, U1.49@16, U1.49@17, U1.49@18, U1.49@2, U1.49@3, U1.49@4, U1.49@5, U1.49@6, U1.49@7, U1.49@8, U1.49@9, U6.4; no longer Q4.2
- net GND2: now also RA1.2, RA1.3, RA2.2, RA2.3, RA3.2, RA3.3, RA4.2, RA4.3, RA5.2, RA5.3, RA5.4; no longer RA1.6, RA1.7, RA2.6, RA2.7, RA3.6, RA3.7, RA4.6, RA4.7, RA5.7
- net GRN1: now also RA9.5; no longer RA9.8
- net GRN2: now also RA8.7; no longer RA8.3
- net GRN3: now also RA8.5; no longer RA8.8
- net GRN4: now also RA9.7; no longer RA9.3
- net K_BSP: now also SW_BSP.1@1, SW_BSP.1@2; no longer SW_BSP.P$1, SW_BSP.P$3
- net K_CL: now also SW_CL.1@1, SW_CL.1@2; no longer SW_CL.P$1, SW_CL.P$3
- net K_DP: now also SW_DP.1@1, SW_DP.1@2; no longer SW_DP.P$1, SW_DP.P$3
- net K_ENT: now also SW_ENT.1@1, SW_ENT.1@2; no longer SW_ENT.P$1, SW_ENT.P$3
- net K_LS: now also SW_LS.1@1, SW_LS.1@2; no longer SW_LS.P$1, SW_LS.P$3
- net LED_PWR_EN: now also U6.3; no longer R73.2
- net N$100: now also SW_N1.1@1, SW_N1.1@2; no longer SW_N1.P$1, SW_N1.P$3
- net N$101: now also SW_N2.1@1, SW_N2.1@2; no longer SW_N2.P$1, SW_N2.P$3
- net N$102: now also SW_N0.1@1, SW_N0.1@2; no longer SW_N0.P$1, SW_N0.P$3
- net N$103: now also SW_RT.1@1, SW_RT.1@2; no longer SW_RT.P$1, SW_RT.P$3
- net N$104: now also SW_DN.1@1, SW_DN.1@2; no longer SW_DN.P$1, SW_DN.P$3
- net N$105: now also SW_LF.1@1, SW_LF.1@2; no longer SW_LF.P$1, SW_LF.P$3
- net N$107: now also SW_RC.1@1, SW_RC.1@2; no longer SW_RC.P$1, SW_RC.P$3
- net N$108: now also SW_RW.1@1, SW_RW.1@2; no longer SW_RW.P$1, SW_RW.P$3
- net N$109: now also SW_RA.1@1, SW_RA.1@2; no longer SW_RA.P$1, SW_RA.P$3
- net N$110: now also SW_SPC.1@1, SW_SPC.1@2; no longer SW_SPC.P$1, SW_SPC.P$3
- net N$111: now also SW_LA.1@1, SW_LA.1@2; no longer SW_LA.P$1, SW_LA.P$3
- net N$112: now also SW_LW.1@1, SW_LW.1@2; no longer SW_LW.P$1, SW_LW.P$3
- net N$113: now also SW_LC.1@1, SW_LC.1@2; no longer SW_LC.P$1, SW_LC.P$3
- net N$114: now also SW_ND.1@1, SW_ND.1@2; no longer SW_ND.P$1, SW_ND.P$3
- net N$115: now also SW_N3.1@1, SW_N3.1@2; no longer SW_N3.P$1, SW_N3.P$3
- net N$116: now also SW_NEN.1@1, SW_NEN.1@2; no longer SW_NEN.P$1, SW_NEN.P$3
- net N$117: now also SW_NP.1@1, SW_NP.1@2; no longer SW_NP.P$1, SW_NP.P$3
- net N$118: now also SW_N9.1@1, SW_N9.1@2; no longer SW_N9.P$1, SW_N9.P$3
- net N$119: now also SW_MIN.1@1, SW_MIN.1@2; no longer SW_MIN.P$1, SW_MIN.P$3
- net N$120: now also SW_MUL.1@1, SW_MUL.1@2; no longer SW_MUL.P$1, SW_MUL.P$3
- net N$121: now also SW_F16.1@1, SW_F16.1@2; no longer SW_F16.P$1, SW_F16.P$3
- net N$123: now also RA7.2; no longer RA7.1
- net N$125: now also RA9.3, U_LED1.21; no longer RA9.4, U_LED1.33
- net N$126: now also RA6.2, U_LED1.20; no longer RA6.4, U_LED1.32
- net N$127: now also RA9.2; no longer RA9.6
- net N$128: now also RA7.4, U_LED1.32; no longer RA9.7, U_LED1.21
- net N$129: now also RA6.3, U_LED1.17; no longer RA6.6, U_LED1.20
- net N$130: now also U_LED1.33; no longer U_LED1.19
- net N$131: now also RA6.4, U_LED1.13; no longer RA6.7, U_LED1.17
- net N$132: now also RA7.3, U_LED1.38; no longer RA8.6, U_LED1.15
- net N$133: now also RA8.3; no longer RA8.7
- net N$134: now also RA8.4, U_LED1.12; no longer RA6.1, U_LED1.13
- net N$135: now also R71.2, U6.6; no longer RA8.1, U_LED1.12
- net N$2: now also SW_N6.1@1, SW_N6.1@2; no longer SW_N6.P$1, SW_N6.P$3
- net N$22: now also RA9.4, U_LED1.19; no longer RA7.7, U_LED1.38
- net N$25: now also SW_ESC.1@1, SW_ESC.1@2; no longer SW_ESC.P$1, SW_ESC.P$3
- net N$26: now also SW_F1.1@1, SW_F1.1@2; no longer SW_F1.P$1, SW_F1.P$3
- net N$27: now also SW_F2.1@1, SW_F2.1@2; no longer SW_F2.P$1, SW_F2.P$3
- net N$28: now also SW_F3.1@1, SW_F3.1@2; no longer SW_F3.P$1, SW_F3.P$3
- net N$29: now also SW_F4.1@1, SW_F4.1@2; no longer SW_F4.P$1, SW_F4.P$3
- net N$30: now also SW_F5.1@1, SW_F5.1@2; no longer SW_F5.P$1, SW_F5.P$3
- net N$31: now also SW_F6.1@1, SW_F6.1@2; no longer SW_F6.P$1, SW_F6.P$3
- net N$32: now also SW_F7.1@1, SW_F7.1@2; no longer SW_F7.P$1, SW_F7.P$3
- net N$33: now also SW_F8.1@1, SW_F8.1@2; no longer SW_F8.P$1, SW_F8.P$3
- net N$34: now also SW_F9.1@1, SW_F9.1@2; no longer SW_F9.P$1, SW_F9.P$3
- net N$35: now also SW_F10.1@1, SW_F10.1@2; no longer SW_F10.P$1, SW_F10.P$3
- net N$36: now also SW_F11.1@1, SW_F11.1@2; no longer SW_F11.P$1, SW_F11.P$3
- net N$37: now also SW_F12.1@1, SW_F12.1@2; no longer SW_F12.P$1, SW_F12.P$3
- net N$38: now also SW_F13.1@1, SW_F13.1@2; no longer SW_F13.P$1, SW_F13.P$3
- net N$39: now also SW_F14.1@1, SW_F14.1@2; no longer SW_F14.P$1, SW_F14.P$3
- net N$40: now also SW_F15.1@1, SW_F15.1@2; no longer SW_F15.P$1, SW_F15.P$3
- net N$41: now also SW_TDL.1@1, SW_TDL.1@2; no longer SW_TDL.P$1, SW_TDL.P$3
- net N$42: now also SW_1.1@1, SW_1.1@2; no longer SW_1.P$1, SW_1.P$3
- net N$43: now also SW_2.1@1, SW_2.1@2; no longer SW_2.P$1, SW_2.P$3
- net N$44: now also SW_3.1@1, SW_3.1@2; no longer SW_3.P$1, SW_3.P$3
- net N$45: now also SW_4.1@1, SW_4.1@2; no longer SW_4.P$1, SW_4.P$3
- net N$46: now also SW_5.1@1, SW_5.1@2; no longer SW_5.P$1, SW_5.P$3
- net N$47: now also SW_6.1@1, SW_6.1@2; no longer SW_6.P$1, SW_6.P$3
- net N$48: now also SW_7.1@1, SW_7.1@2; no longer SW_7.P$1, SW_7.P$3
- net N$49: now also SW_8.1@1, SW_8.1@2; no longer SW_8.P$1, SW_8.P$3
- net N$50: now also SW_9.1@1, SW_9.1@2; no longer SW_9.P$1, SW_9.P$3
- net N$51: now also SW_0.1@1, SW_0.1@2; no longer SW_0.P$1, SW_0.P$3
- net N$52: now also SW_MU.1@1, SW_MU.1@2; no longer SW_MU.P$1, SW_MU.P$3
- net N$53: now also SW_EP.1@1, SW_EP.1@2; no longer SW_EP.P$1, SW_EP.P$3
- net N$55: now also SW_NUM.1@1, SW_NUM.1@2; no longer SW_NUM.P$1, SW_NUM.P$3
- net N$56: now also SW_DSH.1@1, SW_DSH.1@2; no longer SW_DSH.P$1, SW_DSH.P$3
- net N$57: now also SW_Q.1@1, SW_Q.1@2; no longer SW_Q.P$1, SW_Q.P$3
- net N$58: now also SW_TAB.1@1, SW_TAB.1@2; no longer SW_TAB.P$1, SW_TAB.P$3
- net N$59: now also SW_W.1@1, SW_W.1@2; no longer SW_W.P$1, SW_W.P$3
- net N$60: now also SW_E.1@1, SW_E.1@2; no longer SW_E.P$1, SW_E.P$3
- net N$61: now also SW_R.1@1, SW_R.1@2; no longer SW_R.P$1, SW_R.P$3
- net N$62: now also SW_T.1@1, SW_T.1@2; no longer SW_T.P$1, SW_T.P$3
- net N$63: now also SW_Y.1@1, SW_Y.1@2; no longer SW_Y.P$1, SW_Y.P$3
- net N$64: now also SW_U.1@1, SW_U.1@2; no longer SW_U.P$1, SW_U.P$3
- net N$65: now also SW_I.1@1, SW_I.1@2; no longer SW_I.P$1, SW_I.P$3
- net N$66: now also SW_O.1@1, SW_O.1@2; no longer SW_O.P$1, SW_O.P$3
- net N$67: now also SW_P.1@1, SW_P.1@2; no longer SW_P.P$1, SW_P.P$3
- net N$68: now also SW_OB.1@1, SW_OB.1@2; no longer SW_OB.P$1, SW_OB.P$3
- net N$69: now also SW_CB.1@1, SW_CB.1@2; no longer SW_CB.P$1, SW_CB.P$3
- net N$71: now also SW_N7.1@1, SW_N7.1@2; no longer SW_N7.P$1, SW_N7.P$3
- net N$72: now also SW_N8.1@1, SW_N8.1@2; no longer SW_N8.P$1, SW_N8.P$3
- net N$73: now also SW_N5.1@1, SW_N5.1@2; no longer SW_N5.P$1, SW_N5.P$3
- net N$74: now also SW_N4.1@1, SW_N4.1@2; no longer SW_N4.P$1, SW_N4.P$3
- net N$76: now also SW_QU.1@1, SW_QU.1@2; no longer SW_QU.P$1, SW_QU.P$3
- net N$77: now also SW_CS.1@1, SW_CS.1@2; no longer SW_CS.P$1, SW_CS.P$3
- net N$78: now also SW_L.1@1, SW_L.1@2; no longer SW_L.P$1, SW_L.P$3
- net N$80: now also SW_A.1@1, SW_A.1@2; no longer SW_A.P$1, SW_A.P$3
- net N$81: now also SW_S.1@1, SW_S.1@2; no longer SW_S.P$1, SW_S.P$3
- net N$82: now also SW_D.1@1, SW_D.1@2; no longer SW_D.P$1, SW_D.P$3
- net N$83: now also SW_F.1@1, SW_F.1@2; no longer SW_F.P$1, SW_F.P$3
- net N$84: now also SW_G.1@1, SW_G.1@2; no longer SW_G.P$1, SW_G.P$3
- net N$85: now also SW_H.1@1, SW_H.1@2; no longer SW_H.P$1, SW_H.P$3
- net N$86: now also SW_J.1@1, SW_J.1@2; no longer SW_J.P$1, SW_J.P$3
- net N$87: now also SW_K.1@1, SW_K.1@2; no longer SW_K.P$1, SW_K.P$3
- net N$88: now also SW_Z.1@1, SW_Z.1@2; no longer SW_Z.P$1, SW_Z.P$3
- net N$89: now also SW_X.1@1, SW_X.1@2; no longer SW_X.P$1, SW_X.P$3
- net N$90: now also SW_C.1@1, SW_C.1@2; no longer SW_C.P$1, SW_C.P$3
- net N$91: now also SW_V.1@1, SW_V.1@2; no longer SW_V.P$1, SW_V.P$3
- net N$92: now also SW_B.1@1, SW_B.1@2; no longer SW_B.P$1, SW_B.P$3
- net N$93: now also SW_N.1@1, SW_N.1@2; no longer SW_N.P$1, SW_N.P$3
- net N$94: now also SW_M.1@1, SW_M.1@2; no longer SW_M.P$1, SW_M.P$3
- net N$95: now also SW_CM.1@1, SW_CM.1@2; no longer SW_CM.P$1, SW_CM.P$3
- net N$96: now also SW_DT.1@1, SW_DT.1@2; no longer SW_DT.P$1, SW_DT.P$3
- net N$97: now also SW_FS.1@1, SW_FS.1@2; no longer SW_FS.P$1, SW_FS.P$3
- net N$98: now also SW_RS.1@1, SW_RS.1@2; no longer SW_RS.P$1, SW_RS.P$3
- net N$99: now also SW_UP.1@1, SW_UP.1@2; no longer SW_UP.P$1, SW_UP.P$3
- net RED1: now also RA6.7; no longer RA6.3
- net RED2: now also RA6.6; no longer RA6.2
- net RED3: now also RA6.5; no longer RA6.8
- net RED4: now also RA7.5; no longer RA6.5
- net RED5: now also RA7.7; no longer RA7.8
- net RED6: now also RA7.6; no longer RA7.2
- net ROW0: now also SW_ESC.2@1, SW_ESC.2@2, SW_F1.2@1, SW_F1.2@2, SW_F10.2@1, SW_F10.2@2, SW_F11.2@1, SW_F11.2@2, SW_F12.2@1, SW_F12.2@2, SW_F13.2@1, SW_F13.2@2, SW_F14.2@1, SW_F14.2@2, SW_F15.2@1, SW_F15.2@2, SW_F16.2@1, SW_F16.2@2, SW_F2.2@1, SW_F2.2@2, SW_F3.2@1, SW_F3.2@2, SW_F4.2@1, SW_F4.2@2, SW_F5.2@1, SW_F5.2@2, SW_F6.2@1, SW_F6.2@2, SW_F7.2@1, SW_F7.2@2, SW_F8.2@1, SW_F8.2@2, SW_F9.2@1, SW_F9.2@2; no longer SW_ESC.P$2, SW_ESC.P$4, SW_F1.P$2, SW_F1.P$4, SW_F10.P$2, SW_F10.P$4, SW_F11.P$2, SW_F11.P$4, SW_F12.P$2, SW_F12.P$4, SW_F13.P$2, SW_F13.P$4, SW_F14.P$2, SW_F14.P$4, SW_F15.P$2, SW_F15.P$4, SW_F16.P$2, SW_F16.P$4, SW_F2.P$2, SW_F2.P$4, SW_F3.P$2, SW_F3.P$4, SW_F4.P$2, SW_F4.P$4, SW_F5.P$2, SW_F5.P$4, SW_F6.P$2, SW_F6.P$4, SW_F7.P$2, SW_F7.P$4, SW_F8.P$2, SW_F8.P$4, SW_F9.P$2, SW_F9.P$4
- net ROW1: now also SW_0.2@1, SW_0.2@2, SW_1.2@1, SW_1.2@2, SW_2.2@1, SW_2.2@2, SW_3.2@1, SW_3.2@2, SW_4.2@1, SW_4.2@2, SW_5.2@1, SW_5.2@2, SW_6.2@1, SW_6.2@2, SW_7.2@1, SW_7.2@2, SW_8.2@1, SW_8.2@2, SW_9.2@1, SW_9.2@2, SW_BSP.2@1, SW_BSP.2@2, SW_DSH.2@1, SW_DSH.2@2, SW_EP.2@1, SW_EP.2@2, SW_MIN.2@1, SW_MIN.2@2, SW_MU.2@1, SW_MU.2@2, SW_MUL.2@1, SW_MUL.2@2, SW_NUM.2@1, SW_NUM.2@2, SW_TDL.2@1, SW_TDL.2@2; no longer SW_0.P$2, SW_0.P$4, SW_1.P$2, SW_1.P$4, SW_2.P$2, SW_2.P$4, SW_3.P$2, SW_3.P$4, SW_4.P$2, SW_4.P$4, SW_5.P$2, SW_5.P$4, SW_6.P$2, SW_6.P$4, SW_7.P$2, SW_7.P$4, SW_8.P$2, SW_8.P$4, SW_9.P$2, SW_9.P$4, SW_BSP.P$2, SW_BSP.P$4, SW_DSH.P$2, SW_DSH.P$4, SW_EP.P$2, SW_EP.P$4, SW_MIN.P$2, SW_MIN.P$4, SW_MU.P$2, SW_MU.P$4, SW_MUL.P$2, SW_MUL.P$4, SW_NUM.P$2, SW_NUM.P$4, SW_TDL.P$2, SW_TDL.P$4
- net ROW2: now also SW_CB.2@1, SW_CB.2@2, SW_DP.2@1, SW_DP.2@2, SW_E.2@1, SW_E.2@2, SW_I.2@1, SW_I.2@2, SW_N7.2@1, SW_N7.2@2, SW_N8.2@1, SW_N8.2@2, SW_N9.2@1, SW_N9.2@2, SW_NP.2@1, SW_NP.2@2, SW_O.2@1, SW_O.2@2, SW_OB.2@1, SW_OB.2@2, SW_P.2@1, SW_P.2@2, SW_Q.2@1, SW_Q.2@2, SW_R.2@1, SW_R.2@2, SW_T.2@1, SW_T.2@2, SW_TAB.2@1, SW_TAB.2@2, SW_U.2@1, SW_U.2@2, SW_W.2@1, SW_W.2@2, SW_Y.2@1, SW_Y.2@2; no longer SW_CB.P$2, SW_CB.P$4, SW_DP.P$2, SW_DP.P$4, SW_E.P$2, SW_E.P$4, SW_I.P$2, SW_I.P$4, SW_N7.P$2, SW_N7.P$4, SW_N8.P$2, SW_N8.P$4, SW_N9.P$2, SW_N9.P$4, SW_NP.P$2, SW_NP.P$4, SW_O.P$2, SW_O.P$4, SW_OB.P$2, SW_OB.P$4, SW_P.P$2, SW_P.P$4, SW_Q.P$2, SW_Q.P$4, SW_R.P$2, SW_R.P$4, SW_T.P$2, SW_T.P$4, SW_TAB.P$2, SW_TAB.P$4, SW_U.P$2, SW_U.P$4, SW_W.P$2, SW_W.P$4, SW_Y.P$2, SW_Y.P$4
- net ROW3: now also SW_A.2@1, SW_A.2@2, SW_CL.2@1, SW_CL.2@2, SW_CS.2@1, SW_CS.2@2, SW_D.2@1, SW_D.2@2, SW_ENT.2@1, SW_ENT.2@2, SW_F.2@1, SW_F.2@2, SW_G.2@1, SW_G.2@2, SW_H.2@1, SW_H.2@2, SW_J.2@1, SW_J.2@2, SW_K.2@1, SW_K.2@2, SW_L.2@1, SW_L.2@2, SW_N4.2@1, SW_N4.2@2, SW_N5.2@1, SW_N5.2@2, SW_N6.2@1, SW_N6.2@2, SW_QU.2@1, SW_QU.2@2, SW_S.2@1, SW_S.2@2; no longer SW_A.P$2, SW_A.P$4, SW_CL.P$2, SW_CL.P$4, SW_CS.P$2, SW_CS.P$4, SW_D.P$2, SW_D.P$4, SW_ENT.P$2, SW_ENT.P$4, SW_F.P$2, SW_F.P$4, SW_G.P$2, SW_G.P$4, SW_H.P$2, SW_H.P$4, SW_J.P$2, SW_J.P$4, SW_K.P$2, SW_K.P$4, SW_L.P$2, SW_L.P$4, SW_N4.P$2, SW_N4.P$4, SW_N5.P$2, SW_N5.P$4, SW_N6.P$2, SW_N6.P$4, SW_QU.P$2, SW_QU.P$4, SW_S.P$2, SW_S.P$4
- net ROW4: now also SW_B.2@1, SW_B.2@2, SW_C.2@1, SW_C.2@2, SW_CM.2@1, SW_CM.2@2, SW_DT.2@1, SW_DT.2@2, SW_FS.2@1, SW_FS.2@2, SW_LS.2@1, SW_LS.2@2, SW_M.2@1, SW_M.2@2, SW_N.2@1, SW_N.2@2, SW_N1.2@1, SW_N1.2@2, SW_N2.2@1, SW_N2.2@2, SW_N3.2@1, SW_N3.2@2, SW_NEN.2@1, SW_NEN.2@2, SW_RS.2@1, SW_RS.2@2, SW_UP.2@1, SW_UP.2@2, SW_V.2@1, SW_V.2@2, SW_X.2@1, SW_X.2@2, SW_Z.2@1, SW_Z.2@2; no longer SW_B.P$2, SW_B.P$4, SW_C.P$2, SW_C.P$4, SW_CM.P$2, SW_CM.P$4, SW_DT.P$2, SW_DT.P$4, SW_FS.P$2, SW_FS.P$4, SW_LS.P$2, SW_LS.P$4, SW_M.P$2, SW_M.P$4, SW_N.P$2, SW_N.P$4, SW_N1.P$2, SW_N1.P$4, SW_N2.P$2, SW_N2.P$4, SW_N3.P$2, SW_N3.P$4, SW_NEN.P$2, SW_NEN.P$4, SW_RS.P$2, SW_RS.P$4, SW_UP.P$2, SW_UP.P$4, SW_V.P$2, SW_V.P$4, SW_X.P$2, SW_X.P$4, SW_Z.P$2, SW_Z.P$4
- net ROW5: now also SW_DN.2@1, SW_DN.2@2, SW_LA.2@1, SW_LA.2@2, SW_LC.2@1, SW_LC.2@2, SW_LF.2@1, SW_LF.2@2, SW_LW.2@1, SW_LW.2@2, SW_N0.2@1, SW_N0.2@2, SW_ND.2@1, SW_ND.2@2, SW_RA.2@1, SW_RA.2@2, SW_RC.2@1, SW_RC.2@2, SW_RT.2@1, SW_RT.2@2, SW_RW.2@1, SW_RW.2@2, SW_SPC.2@1, SW_SPC.2@2; no longer SW_DN.P$2, SW_DN.P$4, SW_LA.P$2, SW_LA.P$4, SW_LC.P$2, SW_LC.P$4, SW_LF.P$2, SW_LF.P$4, SW_LW.P$2, SW_LW.P$4, SW_N0.P$2, SW_N0.P$4, SW_ND.P$2, SW_ND.P$4, SW_RA.P$2, SW_RA.P$4, SW_RC.P$2, SW_RC.P$4, SW_RT.P$2, SW_RT.P$4, SW_RW.P$2, SW_RW.P$4, SW_SPC.P$2, SW_SPC.P$4
- net USB_DP: now also R46.1
- net VCC_1: now also U6.1, U6.2; no longer Q3.2, R71.2
Routing:
- net ROW1: track 0.00 -> 361.9 mm
- net ROW3: track 0.00 -> 355.5 mm
- net ROW2: track 0.00 -> 352.6 mm
- net ROW4: track 0.00 -> 349.6 mm
- net ROW5: track 0.00 -> 341.1 mm
- net ROW0: track 0.00 -> 335.1 mm
- net VCC_1: track 0.00 -> 50.8 mm
- net VCC_2: track 0.00 -> 40.6 mm
- net Y2I: track 0.00 -> 33.7 mm
- net Y2O: track 0.00 -> 29.0 mm
- net N$119: track 0.00 -> 26.7 mm
- net Y1O: track 0.00 -> 25.3 mm
- net Y1I: track 0.00 -> 24.7 mm
- net N$121: track 0.00 -> 24.6 mm, vias 0 -> 1
- net USB_DP: track 0.00 -> 22.8 mm
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- added copper zone on layer 1, net GND
- added copper zone on layer 16, net GND
Other:
- outline, holes or cut-outs redrawn

Commit message: wip
Parts:
- removed RA1, RA2, RA3, RA4, RA5: 10K, __untitled:R0603X4
- removed RA10, RA13, RA14, RA15, RA8, RA9: 20R, __untitled:R0603X4
- removed RA11, RA12, RA6, RA7: 51R, __untitled:R0603X4
- added R1, R2, R3, R4, R5: 10K, ts_keyboards:R0603X4
- added R10, R11, R6, R7, R8, R9: 20R, ts_keyboards:R0603X4
- added R12, R13, R14, R15: 51R, ts_keyboards:R0603X4
- R41, R42: value (none) -> 4K7
- moved R38 221.3 mm to (30.5, 58.0), turned to 90 degrees
- moved C4 214.9 mm to (20.0, 61.0), turned to 180 degrees
- moved C5 214.6 mm to (33.0, 59.0)
- moved C2 210.3 mm to (33.0, 61.0)
- moved R37 206.5 mm to (33.0, 57.0)
- moved C3 206.2 mm to (20.0, 63.0), turned to 180 degrees
- moved C1 197.2 mm to (33.0, 63.0)
- moved C10 81.5 mm to (104.5, 102.0)
- moved C9 81.5 mm to (128.8, 103.0)
- moved R39 81.5 mm to (123.1, 103.0)
- moved C6 81.5 mm to (109.1, 102.7)
- moved C7 81.5 mm to (135.2, 103.0)
- moved C8 81.5 mm to (113.0, 102.7)
- moved R40 81.5 mm to (117.7, 102.7)
- moved D55 11.0 mm to (26.0, 45.0)
Connections:
- removed net N$10: RA12.4, U_LED2.32
- removed net N$11: RA14.6, U_LED2.31
- removed net N$12: RA14.7, U_LED2.21
- removed net N$122: RA8.2, U_LED1.15
- removed net N$123: RA7.2, U_LED1.35
- removed net N$124: RA10.1, U_LED1.34
- removed net N$125: RA9.3, U_LED1.21
- removed net N$126: RA6.2, U_LED1.20
- removed net N$127: RA9.2, U_LED1.31
- removed net N$128: RA7.4, U_LED1.32
- removed net N$129: RA6.3, U_LED1.17
- removed net N$13: RA12.6, U_LED2.20
- removed net N$130: RA9.1, U_LED1.33
- removed net N$131: RA6.4, U_LED1.13
- removed net N$132: RA7.3, U_LED1.38
- removed net N$133: RA8.3, U_LED1.14
- removed net N$134: RA8.4, U_LED1.12
- removed net N$14: RA14.1, U_LED2.19
- removed net N$15: RA12.7, U_LED2.17
- removed net N$16: RA13.6, U_LED2.15
- removed net N$17: RA13.7, U_LED2.14
- removed net N$18: RA12.1, U_LED2.13
- removed net N$19: RA13.1, U_LED2.12
- removed net N$20: RA13.4, U_LED2.18
- removed net N$21: RA10.4, U_LED1.39
- removed net N$22: RA9.4, U_LED1.19
- removed net N$23: RA10.6, U_LED1.37
- removed net N$24: RA10.7, U_LED1.36
- removed net N$3: RA15.4, U_LED2.39
- removed net N$4: RA11.7, U_LED2.38
- removed net N$5: RA15.6, U_LED2.37
- removed net N$6: RA15.7, U_LED2.36
- removed net N$7: RA11.1, U_LED2.35
- removed net N$79: RA8.1, U_LED1.18
- removed net N$8: RA15.1, U_LED2.34
- removed net N$9: RA14.4, U_LED2.33
- new net XB1: R6.1, U_LED1.39
- new net XB10: R10.3, U_LED2.21
- new net XB11: R11.1, U_LED2.18
- new net XB12: R11.3, U_LED2.14
- new net XB2: R6.3, U_LED1.36
- new net XB3: R7.1, U_LED1.33
- new net XB4: R7.3, U_LED1.21
- new net XB5: R8.1, U_LED1.18
- new net XB6: R8.3, U_LED1.14
- new net XB7: R9.1, U_LED2.39
- new net XB8: R9.3, U_LED2.36
- new net XB9: R10.1, U_LED2.33
- new net XG1: R6.2, U_LED1.38
- new net XG10: R10.4, U_LED2.20
- new net XG11: R11.2, U_LED2.17
- new net XG12: R11.4, U_LED2.13
- new net XG2: R6.4, U_LED1.35
- new net XG3: R7.2, U_LED1.32
- new net XG4: R7.4, U_LED1.20
- new net XG5: R8.2, U_LED1.17
- new net XG6: R8.4, U_LED1.13
- new net XG7: R9.2, U_LED2.38
- new net XG8: R9.4, U_LED2.35
- new net XG9: R10.2, U_LED2.32
- new net XR1: R12.1, U_LED1.37
- new net XR10: R15.1, U_LED2.19
- new net XR11: R15.2, U_LED2.15
- new net XR12: R15.3, U_LED2.12
- new net XR2: R12.2, U_LED1.34
- new net XR3: R12.3, U_LED1.31
- new net XR4: R13.1, U_LED1.19
- new net XR5: R13.2, U_LED1.15
- new net XR6: R13.3, U_LED1.12
- new net XR7: R14.1, U_LED2.37
- new net XR8: R14.2, U_LED2.34
- new net XR9: R14.3, U_LED2.31
- net BLU1: now also R6.8; no longer RA9.6
- net BLU10: now also R10.6; no longer RA14.5
- net BLU11: now also R11.8; no longer RA15.2
- net BLU12: now also R11.6; no longer RA15.5
- net BLU2: now also R6.6; no longer RA8.8
- net BLU3: now also R7.8; no longer RA8.6
- net BLU4: now also R7.6; no longer RA9.8
- net BLU5: now also R8.8; no longer RA10.2
- net BLU6: now also R8.6; no longer RA10.5
- net BLU7: now also R9.8; no longer RA14.2
- net BLU8: now also R9.6; no longer RA13.5
- net BLU9: now also R10.8; no longer RA13.2
- net COL0: now also R4.8; no longer RA4.8
- net COL1: now also R4.7; no longer RA4.7
- net COL10: now also R2.5; no longer RA2.5
- net COL11: now also R3.8; no longer RA3.8
- net COL12: now also R3.7; no longer RA3.7
- net COL13: now also R3.6; no longer RA3.6
- net COL14: now also R1.8; no longer RA1.8
- net COL15: now also R1.7; no longer RA1.7
- net COL16: now also R1.6; no longer RA1.6
- net COL17: now also R1.5; no longer RA1.5
- net COL2: now also R4.6; no longer RA4.6
- net COL3: now also R4.5; no longer RA4.5
- net COL4: now also R5.8; no longer RA5.8
- net COL5: now also R5.7; no longer RA5.7
- net COL6: now also R5.6; no longer RA5.6
- net COL7: now also R2.8; no longer RA2.8
- net COL8: now also R2.7; no longer RA2.7
- net COL9: now also R2.6; no longer RA2.6
- net GND2: now also R1.1, R1.2, R1.3, R1.4, R2.1, R2.2, R2.3, R2.4, R3.1, R3.2, R3.3, R4.1, R4.2, R4.3, R4.4, R5.1, R5.2, R5.3; no longer RA1.1, RA1.2, RA1.3, RA1.4, RA2.1, RA2.2, RA2.3, RA2.4, RA3.1, RA3.2, RA3.3, RA3.4, RA4.1, RA4.2, RA4.3, RA4.4, RA5.1, RA5.2, RA5.3, RA5.4
- net GRN1: now also R6.7; no longer RA9.5
- net GRN10: now also R10.5; no longer RA14.3
- net GRN11: now also R11.7; no longer RA15.8
- net GRN12: now also R11.5; no longer RA15.3
- net GRN2: now also R6.5; no longer RA8.7
- net GRN3: now also R7.7; no longer RA8.5
- net GRN4: now also R7.5; no longer RA9.7
- net GRN5: now also R8.7; no longer RA10.8
- net GRN6: now also R8.5; no longer RA10.3
- net GRN7: now also R9.7; no longer RA14.8
- net GRN8: now also R9.5; no longer RA13.3
- net GRN9: now also R10.7; no longer RA13.8
- net RED1: now also R12.8; no longer RA6.7
- net RED10: now also R15.8; no longer RA12.5
- net RED11: now also R15.7; no longer RA11.8
- net RED12: now also R15.6; no longer RA11.2
- net RED2: now also R12.7; no longer RA6.6
- net RED3: now also R12.6; no longer RA6.5
- net RED4: now also R13.8; no longer RA7.5
- net RED5: now also R13.7; no longer RA7.7
- net RED6: now also R13.6; no longer RA7.6
- net RED7: now also R14.8; no longer RA12.3
- net RED8: now also R14.7; no longer RA12.2
- net RED9: now also R14.6; no longer RA12.8
Routing:
- net VCC_LED: track 0.00 -> 11.2 mm
- net N$131: track 10.8 -> 0.00 mm, vias 2 -> 0
- net N$129: track 9.62 -> 0.00 mm, vias 2 -> 0
- net ROW3: track 355.5 -> 346.4 mm
- net LED_SBD: track 0.00 -> 8.48 mm
- net N$133: track 8.47 -> 0.00 mm
- net N$122: track 8.47 -> 0.00 mm
- net N$134: track 8.25 -> 0.00 mm
- net N$79: track 8.00 -> 0.00 mm
- net K_CL: track 7.64 -> 1.00 mm
- net VCC_2: track 40.6 -> 38.0 mm
