File: EAGLE/vr98/vr98-revA.sch (EAGLE design)
At the start: 405 parts, among them Q1 2N7002, Q2 DMG2305UX-7, U1 STM32F411CEU7THERM, U2 74HC589A_DT, U3 74HC589A_DT, U4 74HC589A_DT, U5 M25C, U6 TPS22995H-Q1, Y1 32.768kHz ±20ppm 6pF, Y2 25MHz 9pF

Commit message: wip
Parts:
- removed RA1, RA2, RA3, RA4, RA5: 10K, __untitled:R-EU-4_
- removed RA10, RA13, RA14, RA15, RA8, RA9: 20R, __untitled:R-EU-4_
- removed RA11, RA12, RA6, RA7: 51R, __untitled:R-EU-4_
- added R1, R2, R3, R4, R5: 10K, ts_keyboards:R-EU-4
- added R10, R11, R6, R7, R8, R9: 20R, ts_keyboards:R-EU-4
- added R12, R13, R14, R15: 51R, ts_keyboards:R-EU-4
- R41, R42: value (none) -> 4K7
Connections:
- removed net N$10: RA12D.1, U_LED2.CS8
- removed net N$11: RA14C.2, U_LED2.CS9
- removed net N$12: RA14B.2, U_LED2.CS10
- removed net N$122: RA8B.1, U_LED1.CS15
- removed net N$123: RA7B.1, U_LED1.CS5
- removed net N$124: RA10A.1, U_LED1.CS6
- removed net N$125: RA9C.1, U_LED1.CS10
- removed net N$126: RA6B.1, U_LED1.CS11
- removed net N$127: RA9B.1, U_LED1.CS9
- removed net N$128: RA7D.1, U_LED1.CS8
- removed net N$129: RA6C.1, U_LED1.CS14
- removed net N$13: RA12C.2, U_LED2.CS11
- removed net N$130: RA9A.1, U_LED1.CS7
- removed net N$131: RA6D.1, U_LED1.CS17
- removed net N$132: RA7C.1, U_LED1.CS2
- removed net N$133: RA8C.1, U_LED1.CS16
- removed net N$134: RA8D.1, U_LED1.CS18
- removed net N$14: RA14A.1, U_LED2.CS12
- removed net N$15: RA12B.2, U_LED2.CS14
- removed net N$16: RA13C.2, U_LED2.CS15
- removed net N$17: RA13B.2, U_LED2.CS16
- removed net N$18: RA12A.1, U_LED2.CS17
- removed net N$19: RA13A.1, U_LED2.CS18
- removed net N$20: RA13D.1, U_LED2.CS13
- removed net N$21: RA10D.1, U_LED1.CS1
- removed net N$22: RA9D.1, U_LED1.CS12
- removed net N$23: RA10C.2, U_LED1.CS3
- removed net N$24: RA10B.2, U_LED1.CS4
- removed net N$3: RA15D.1, U_LED2.CS1
- removed net N$4: RA11B.2, U_LED2.CS2
- removed net N$5: RA15C.2, U_LED2.CS3
- removed net N$6: RA15B.2, U_LED2.CS4
- removed net N$7: RA11A.1, U_LED2.CS5
- removed net N$79: RA8A.1, U_LED1.CS13
- removed net N$8: RA15A.1, U_LED2.CS6
- removed net N$9: RA14D.1, U_LED2.CS7
- new net XB1: R6.1, U_LED1.CS1
- new net XB10: R10.3, U_LED2.CS10
- new net XB11: R11.1, U_LED2.CS13
- new net XB12: R11.3, U_LED2.CS16
- new net XB2: R6.3, U_LED1.CS4
- new net XB3: R7.1, U_LED1.CS7
- new net XB4: R7.3, U_LED1.CS10
- new net XB5: R8.1, U_LED1.CS13
- new net XB6: R8.3, U_LED1.CS16
- new net XB7: R9.1, U_LED2.CS1
- new net XB8: R9.3, U_LED2.CS4
- new net XB9: R10.1, U_LED2.CS7
- new net XG1: R6.2, U_LED1.CS2
- new net XG10: R10.4, U_LED2.CS11
- new net XG11: R11.2, U_LED2.CS14
- new net XG12: R11.4, U_LED2.CS17
- new net XG2: R6.4, U_LED1.CS5
- new net XG3: R7.2, U_LED1.CS8
- new net XG4: R7.4, U_LED1.CS11
- new net XG5: R8.2, U_LED1.CS14
- new net XG6: R8.4, U_LED1.CS17
- new net XG7: R9.2, U_LED2.CS2
- new net XG8: R9.4, U_LED2.CS5
- new net XG9: R10.2, U_LED2.CS8
- new net XR1: R12.1, U_LED1.CS3
- new net XR10: R15.1, U_LED2.CS12
- new net XR11: R15.2, U_LED2.CS15
- new net XR12: R15.3, U_LED2.CS18
- new net XR2: R12.2, U_LED1.CS6
- new net XR3: R12.3, U_LED1.CS9
- new net XR4: R13.1, U_LED1.CS12
- new net XR5: R13.2, U_LED1.CS15
- new net XR6: R13.3, U_LED1.CS18
- new net XR7: R14.1, U_LED2.CS3
- new net XR8: R14.2, U_LED2.CS6
- new net XR9: R14.3, U_LED2.CS9
- net BLU1: now also R6.8; no longer RA9C.2
- net BLU10: now also R10.6; no longer RA14D.2
- net BLU11: now also R11.8; no longer RA15B.1
- net BLU12: now also R11.6; no longer RA15D.2
- net BLU2: now also R6.6; no longer RA8A.2
- net BLU3: now also R7.8; no longer RA8C.2
- net BLU4: now also R7.6; no longer RA9A.2
- net BLU5: now also R8.8; no longer RA10B.1
- net BLU6: now also R8.6; no longer RA10D.2
- net BLU7: now also R9.8; no longer RA14B.1
- net BLU8: now also R9.6; no longer RA13D.2
- net BLU9: now also R10.8; no longer RA13B.1
- net COL0: now also R4.8; no longer RA4A.2
- net COL1: now also R4.7; no longer RA4B.2
- net COL10: now also R2.5; no longer RA2D.2
- net COL11: now also R3.8; no longer RA3A.2
- net COL12: now also R3.7; no longer RA3B.2
- net COL13: now also R3.6; no longer RA3C.2
- net COL14: now also R1.8; no longer RA1A.2
- net COL15: now also R1.7; no longer RA1B.2
- net COL16: now also R1.6; no longer RA1C.2
- net COL17: now also R1.5; no longer RA1D.2
- net COL2: now also R4.6; no longer RA4C.2
- net COL3: now also R4.5; no longer RA4D.2
- net COL4: now also R5.8; no longer RA5A.2
- net COL5: now also R5.7; no longer RA5B.2
- net COL6: now also R5.6; no longer RA5C.2
- net COL7: now also R2.8; no longer RA2A.2
- net COL8: now also R2.7; no longer RA2B.2
- net COL9: now also R2.6; no longer RA2C.2
- net GND2: now also R1.1, R1.2, R1.3, R1.4, R2.1, R2.2, R2.3, R2.4, R3.1, R3.2, R3.3, R4.1, R4.2, R4.3, R4.4, R5.1, R5.2, R5.3; no longer RA1A.1, RA1B.1, RA1C.1, RA1D.1, RA2A.1, RA2B.1, RA2C.1, RA2D.1, RA3A.1, RA3B.1, RA3C.1, RA3D.1, RA4A.1, RA4B.1, RA4C.1, RA4D.1, RA5A.1, RA5B.1, RA5C.1, RA5D.1
- net GRN1: now also R6.7; no longer RA9D.2
- net GRN10: now also R10.5; no longer RA14C.1
- net GRN11: now also R11.7; no longer RA15A.2
- net GRN12: now also R11.5; no longer RA15C.1
- net GRN2: now also R6.5; no longer RA8B.2
- net GRN3: now also R7.7; no longer RA8D.2
- net GRN4: now also R7.5; no longer RA9B.2
- net GRN5: now also R8.7; no longer RA10A.2
- net GRN6: now also R8.5; no longer RA10C.1
- net GRN7: now also R9.7; no longer RA14A.2
- net GRN8: now also R9.5; no longer RA13C.1
- net GRN9: now also R10.7; no longer RA13A.2
- net RED1: now also R12.8; no longer RA6B.2
- net RED10: now also R15.8; no longer RA12D.2
- net RED11: now also R15.7; no longer RA11A.2
- net RED12: now also R15.6; no longer RA11B.1
- net RED2: now also R12.7; no longer RA6C.2
- net RED3: now also R12.6; no longer RA6D.2
- net RED4: now also R13.8; no longer RA7D.2
- net RED5: now also R13.7; no longer RA7B.2
- net RED6: now also R13.6; no longer RA7C.2
- net RED7: now also R14.8; no longer RA12C.1
- net RED8: now also R14.7; no longer RA12B.1
- net RED9: now also R14.6; no longer RA12A.2
Other:
- note added: "DNP / Not Used I2C Pull-up"
- note removed: "I2C Pull-up"
- moved on the sheet: C1, C10, C2, C25, C26, C27, C29, C3, C4, C5, C6, C7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
