File: EAGLE/vr98/vr98-north-revA.brd (EAGLE design)
At the start: 369.5 x 121.8 mm, 405 parts, among them Q1 2N7002, Q2 DMG2305UX-7, U1 STM32F411CEU7THERM, U2 74HC589A_DT, U3 74HC589A_DT, U4 74HC589A_DT, U5 M25C, U6 TPS22995H-Q1, Y1 32.768kHz ±20ppm 6pF, Y2 25MHz 9pF

Commit message: parking the north variant for now
Parts:
- removed R43, R44: 5.1K, rcl:R0603
- removed U$3, U$4: MOLEX_0781710006, molex-pico-ezmate:MOLEX_781710006
- added J2: (no value), molex-pico-ezmate:MOLEX_781710004
- added R16, R17: 5.1K, rcl:R0603
- added SW_CL2: MX-5-PIN-MILMAX-3305-XNO-SILK, ts_keyboards:MX-5-PIN-MILMAX-3305-X-NS
- added U$1, U$2: MOLEX_0781710006, molex-pico-ezmate:MOLEX_781710006
- moved UDB2 81.8 mm to (328.8, 103.0)
- moved UDB1 81.6 mm to (325.0, 103.0)
- moved JKEY 71.8 mm to (24.0, 103.0), turned to 270 degrees
- moved R1 64.0 mm to (273.0, 102.0)
- moved C27 54.0 mm to (273.0, 105.0)
- moved U4 51.0 mm to (278.0, 103.0)
- moved R46 45.3 mm to (312.4, 101.3)
- moved R45 45.0 mm to (312.4, 104.3)
- moved R65 37.0 mm to (283.1, 101.8)
- moved Q1 32.1 mm to (283.0, 105.0)
- moved D18 29.4 mm to (364.2, 70.2)
- moved D101 24.4 mm to (47.0, 2.00)
- moved D102 24.4 mm to (51.0, 2.00)
- moved D87 15.8 mm to (359.6, 32.3)
- moved D54 15.6 mm to (359.7, 70.2)
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Connections:
- removed net CK/DATA/PWM: JPWM.3, U1.29
- removed net WKUP: U1.10
- new net PA0/WKUP: JPWM.3, U1.10
- new net PA8/UNUSED: U1.29
- net BLU7: now also J2.4
- net ENC_A: now also R16.2, U$2.5; no longer R43.1, U$3.6
- net ENC_B: now also R17.2, U$2.6; no longer R44.1, U$3.5
- net GND: now also U$1.1, U$2.1; no longer U$3.1, U$3.NC1, U$3.NC2, U$4.1, U$4.NC1, U$4.NC2
- net GRN7: now also J2.2
- net K_CL: now also SW_CL2.2
- net LED20: now also J2.1
- net N$106: now also U$1.3; no longer U$4.3
- net N$142: now also U$1.4; no longer U$4.4
- net N$152: now also U$1.5; no longer U$4.5
- net N$154: now also U$1.6; no longer U$4.6
- net N$157: now also U$2.4; no longer U$3.4
- net RED7: now also J2.3
- net ROW0: now also U$2.3; no longer U$3.3
- net ROW3: now also SW_CL2.1
- net VCC_2: now also R16.1, R17.1, U$2.2; no longer R43.2, R44.2, U$3.2
Routing:
- net ROW1: track 361.9 -> 0.00 mm
- net ROW2: track 352.6 -> 0.00 mm
- net ROW4: track 349.6 -> 0.00 mm
- net ROW3: track 346.4 -> 0.00 mm
- net ROW5: track 341.1 -> 0.00 mm
- net ROW0: track 335.1 -> 0.00 mm
- net VCC_1: track 50.8 -> 0.00 mm
- net VCC_2: track 38.0 -> 0.00 mm
- net Y2I: track 33.7 -> 0.00 mm
- net Y2O: track 29.0 -> 0.00 mm
- net N$119: track 26.7 -> 0.00 mm
- net Y1O: track 25.3 -> 0.00 mm
- net Y1I: track 24.7 -> 0.00 mm
- net N$121: track 24.6 -> 0.00 mm, vias 1 -> 0
- net USB_DP: track 22.8 -> 0.00 mm
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Other:
- outline, holes or cut-outs redrawn
- board text added: "DIP SW"
- board text added: "KNOB"
- board text added: "LED"
- board text added: "USB UDB"
