File: EAGLE/vr98/vr98-north-revA.sch (EAGLE design)
At the start: 405 parts, among them Q1 2N7002, Q2 DMG2305UX-7, U1 STM32F411CEU7THERM, U2 74HC589A_DT, U3 74HC589A_DT, U4 74HC589A_DT, U5 M25C, U6 TPS22995H-Q1, Y1 32.768kHz ±20ppm 6pF, Y2 25MHz 9pF

Commit message: parking the north variant for now
Parts:
- removed R43, R44: 5.1K, rcl:R-EU_R0603
- removed U$3, U$4: MOLEX_0781710006, molex-pico-ezmate:MOLEX_0781710006
- added J2: (no value), molex-pico-ezmate:MOLEX_0781710004
- added R16, R17: 5.1K, rcl:R-EU_R0603
- added SW_CL2: MX-5-PIN-MILMAX-3305-XNO-SILK, ts_keyboards:MX-5-PIN-MILMAX-3305-XNO-SILK
- added U$1, U$2: MOLEX_0781710006, molex-pico-ezmate:MOLEX_0781710006
Connections:
- removed net CK/DATA/PWM: JPWM.3, U1A.PA8
- removed net WKUP: U1A.PA0-WKUP
- new net PA0/WKUP: JPWM.3, U1A.PA0-WKUP
- new net PA8/UNUSED: U1A.PA8
- net BLU7: now also J2.4
- net ENC_A: now also R16.2, U$2.5; no longer R43.1, U$3.6
- net ENC_B: now also R17.2, U$2.6; no longer R44.1, U$3.5
- net GND: now also U$1.1, U$2.1; no longer U$3.1, U$3.M, U$4.1, U$4.M
- net GRN7: now also J2.2
- net K_CL: now also SW_CL2.S
- net LED20: now also J2.1
- net N$106: now also U$1.3; no longer U$4.3
- net N$142: now also U$1.4; no longer U$4.4
- net N$152: now also U$1.5; no longer U$4.5
- net N$154: now also U$1.6; no longer U$4.6
- net N$157: now also U$2.4; no longer U$3.4
- net RED7: now also J2.3
- net ROW0: now also U$2.3; no longer U$3.3
- net ROW3: now also SW_CL2.P
- net VCC_2: now also R16.1, R17.1, U$2.2; no longer R43.2, R44.2, U$3.2
Other:
- moved on the sheet: D101, D102, JKEY, JTAG, SW_F17
