File: EAGLE/vr99/vr99-south-revA.brd (EAGLE design)
At the start: 369.5 x 121.8 mm, 405 parts, among them Q1 2N7002, Q2 DMG2305UX-7, U1 STM32F411CEU7THERM, U2 74HC589A_DT, U3 74HC589A_DT, U4 74HC589A_DT, U5 M25C, U6 TPS22995H-Q1, Y1 32.768kHz ±20ppm 6pF, Y2 25MHz 9pF

Commit message: .
Parts:
- added C31, C32: 100nF, rcl:C0603
- added FET1, FET2: AO3401A, __untitled:SOT-23-3L_AOS
- added R0, R19: 10K, rcl:R0603
- R18: value 5.1K -> 10K
- moved C6 146.3 mm to (252.1, 133.7)
- moved C10 140.7 mm to (241.5, 134.0)
- moved C8 137.5 mm to (247.0, 133.7)
- moved D102 136.4 mm to (89.0, 133.0)
- moved D101 136.1 mm to (84.0, 133.0)
- moved R12 134.4 mm to (65.0, 133.0)
- moved R13 134.4 mm to (70.0, 133.0)
- moved R6 134.4 mm to (48.0, 133.0)
- moved R7 134.4 mm to (54.0, 133.0)
- moved R8 134.4 mm to (59.0, 133.0)
- moved R10 133.2 mm to (273.0, 130.0)
- moved R11 133.2 mm to (279.0, 130.0)
- moved R14 133.2 mm to (284.0, 130.0)
- moved R15 133.2 mm to (289.0, 130.0)
- moved R9 133.2 mm to (267.0, 130.0)
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Connections:
- removed net ENC_S: R18.2, SW_F13.S, SW_F17.S, U1.29
- removed net N$144: D101.A, JKEY.3
- removed net N$38: D14.A, SW_F13.1@1, SW_F13.1@2
- removed net ROW6: SW_A.2@1, SW_A.2@2, SW_CL.2@1, SW_CL.2@2, SW_CS.2@1, SW_CS.2@2, SW_D.2@1, SW_D.2@2, SW_ENT.2@1, SW_ENT.2@2, SW_F.2@1, SW_F.2@2, SW_G.2@1, SW_G.2@2, SW_H.2@1, SW_H.2@2, SW_J.2@1, SW_J.2@2, SW_K.2@1, SW_K.2@2, SW_L.2@1, SW_L.2@2, SW_N4.2@1, SW_N4.2@2, SW_N5.2@1, SW_N5.2@2, SW_N6.2@1, SW_N6.2@2, SW_QU.2@1, SW_QU.2@2, SW_S.2@1, SW_S.2@2
- new net COL_G1: R5.5, U2.15
- new net COL_G2: R0.2, U4.15, U4.5, U4.6, U4.7
- new net N$3: FET1.1, R18.1, SW_F13.S
- new net N$5: FET2.1, R19.1, SW_F17.S
- new net S13: D14.A, FET1.3, SW_F13.1@1, SW_F13.1@2
- new net S17: D18.A, FET2.3, SW_F17.1@1, SW_F17.1@2
- net ENC_A: now also C31.1
- net ENC_B: now also C32.1, R17.1; no longer R17.2
- net GND: now also C31.2, C32.2; no longer U2.15, U4.15, U4.5, U4.6, U4.7
- net GND2: now also R0.1, R5.4
- net N$4: now also D101.A, JKEY.4; no longer D18.A, SW_F17.1@1, SW_F17.1@2
- net ROW0: now also FET1.2, FET2.2
- net ROW3: now also JKEY.2, SW_A.2@1, SW_A.2@2, SW_CL.2@1, SW_CL.2@2, SW_CS.2@1, SW_CS.2@2, SW_D.2@1, SW_D.2@2, SW_ENT.2@1, SW_ENT.2@2, SW_F.2@1, SW_F.2@2, SW_G.2@1, SW_G.2@2, SW_H.2@1, SW_H.2@2, SW_J.2@1, SW_J.2@2, SW_K.2@1, SW_K.2@2, SW_L.2@1, SW_L.2@2, SW_N4.2@1, SW_N4.2@2, SW_N5.2@1, SW_N5.2@2, SW_N6.2@1, SW_N6.2@2, SW_QU.2@1, SW_QU.2@2, SW_S.2@1, SW_S.2@2
- net ROW5: now also JKEY.3; no longer JKEY.2, JKEY.4
- net VCC_2: now also R17.2, R18.2, R19.2; no longer R17.1, R18.1
Other:
- board text removed: "KNOB"
- board text removed: "LED"

Commit message: .
Parts:
- removed D201, D202: 1N4148, adafruit:SOT23-R
- removed FET1, FET2: AO3401A, __untitled:SOT-23-3L_AOS
- removed Q1: 2N7002, adafruit:SOT23
- removed Q2: DMG2305UX-7, SparkFun-DiscreteSemi:SOT23-3
- removed R67, R68: 100K, rcl:R0603
- removed R69: /DNP/, rcl:R0603
- removed U5: M25C, ts_kb_mcu:8-SOIC
- added D100: (no value), jlcpcb_basic_parts:SOD-123
- added EEP: M25C, ts_kb_mcu:8-SOIC
- added M_M2: SM05B-SRSS-TB(LF)(SN), __temp_to_delete:CONN5_SM05B-SRSS_JST
- added R20: 100R, rcl:R0603
- added R21: 330K, rcl:R0603
- added R22: 1M, rcl:R0603
- added T0: 2N7002, adafruit:SOT23
- added T1: DTC123JKAT146, __temp_to_delete:TRANS_DTA113TKAT_ROM
- added T2, T3: AO3401A, __untitled:SOT-23-3L_AOS
- C20: value 100nF -> 22uF
- C22: value 22uF -> 100nF
- C29: value (none) -> 10uF; device rcl:C0603 -> rcl:C0805
- JPWM: device SparkFun-Connectors:1X04 -> SparkFun-Connectors:1X05_NO_SILK
- JTAG: value DNP -> CORTEX_JTAG_DEBUG_PTH_NS; device SparkFun-Connectors:2X5_NOSILK -> SparkFun-Connectors:2X5-PTH-1.27MM-NO_SILK
- R0: device rcl:R0603 -> ts_keyboards:R0603X4
- Y2: device SparkFun-Clocks:CRYSTAL-SMD-5X3.2-4PAD -> __temp_to_delete:CRYSTAL_2.5X2
- moved R0 248.6 mm to (325.0, 105.0), turned to 270 degrees
- moved D00 156.3 mm to (151.7, 100.9), turned to 180 degrees
- moved LM1117 142.6 mm to (159.0, 104.0), turned to 270 degrees
- moved C24 140.4 mm to (152.4, 102.7), turned to 0 degrees
- moved C22 135.7 mm to (152.4, 105.7), turned to 0 degrees
- moved C23 122.6 mm to (152.4, 104.2), turned to 0 degrees
- moved R71 119.6 mm to (158.5, 128.7)
- moved C20 117.3 mm to (168.0, 104.0), turned to 90 degrees
- moved C21 115.4 mm to (165.0, 104.0), turned to 90 degrees
- moved U6 114.0 mm to (165.0, 129.0)
- moved R18 92.1 mm to (266.9, 106.8), turned to 270 degrees
- moved J_5V 91.6 mm to (173.9, 128.7)
- moved UDB1 80.3 mm to (185.7, 102.0), turned to 180 degrees
- moved R16 77.4 mm to (290.0, 110.5), turned to 180 degrees
- moved UDB2 77.0 mm to (343.8, 103.0)
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- renumbered J1 to RST
Connections:
- net N$140 renamed USB_N
- net N$141 renamed USB_P
- removed net !BOOT: C30.1, D202.1, Q2.1, R67.1
- removed net COL_G1: R5.5, U2.15
- removed net COL_G2: R0.2, U4.15, U4.5, U4.6, U4.7
- removed net LED_SDB: U1.41
- removed net N$3: FET1.1, R18.1, SW_F13.S
- removed net N$5: FET2.1, R19.1, SW_F17.S
- removed net RESET: D201.3, D202.3, RST.2, S1.3, S1.4
- removed net USB_DN: R45.1, UDB1.2, UDB2.2
- removed net USB_DP: R46.1, UDB1.3, UDB2.3
- new net G1: R4.8, U2.15
- new net G2: R2.8, U3.15
- new net G3: R1.8, U4.15
- new net G4: R0.7, U4.5
- new net G5: R0.6, U4.6
- new net G6: R0.5, U4.7
- new net N$11: D100.A, RST.2, S1.3, S1.4, T1.2
- new net N$6: R19.1, SW_F17.S, T3.1
- new net N$7: R20.1, T1.1
- new net N$8: R18.1, SW_F13.S, T2.1
- new net N$9: D100.C, R21.2
- new net PA8: JPWM.4, U1.29
- new net USB_D_N: M_M2.3, R45.1, UDB1.2, UDB2.2
- new net USB_D_P: M_M2.4, R46.1, UDB1.3, UDB2.3
- net !RESET: now also C30.1, R20.2; no longer C29.2, D201.1, R69.1
- net BLU10: no longer Z103.2
- net BLU8: now also Z102.2
- net BLU9: now also Z103.2; no longer Z102.2
- net BOOT0: now also C29.1, R21.1, R22.1; no longer Q2.3, R68.1
- net COL0: now also R4.7; no longer R4.8
- net COL1: now also R4.6; no longer R4.7
- net COL10: now also R3.8; no longer R2.5
- net COL11: now also R3.7; no longer R3.8
- net COL12: now also R3.6; no longer R3.7
- net COL13: now also R3.5; no longer R3.6
- net COL14: now also R1.7; no longer R1.8
- net COL15: now also R1.6; no longer R1.7
- net COL16: now also R1.5; no longer R1.6
- net COL17: now also R0.8; no longer R1.5
- net COL2: now also R4.5; no longer R4.6
- net COL3: now also R5.8; no longer R4.5
- net COL4: now also R5.7; no longer R5.8
- net COL5: now also R5.6; no longer R5.7
- net COL6: now also R5.5; no longer R5.6
- net COL7: now also R2.7; no longer R2.8
- net COL8: now also R2.6; no longer R2.7
- net COL9: now also R2.5; no longer R2.6
- net EE_CS: now also EEP.1; no longer U5.1
- net GND: now also C29.2, EEP.4, JPWM.5, JTAG.7, M_M2.1, M_M2.2, M_M2.6, M_M2.7, R22.2, T1.3, Y2.2, Y2.4; no longer C29.1, JPWM.4, R68.2, RST.1, S1.1, S1.2, U3.15, U5.4
- net GND2: now also R0.2, R0.3, R0.4, R3.4
- net GRN10: no longer Z103.4
- net GRN8: now also Z102.4
- net GRN9: now also Z103.4; no longer Z102.4
- net LATCH: now also T0.3; no longer Q1.3
- net LED15: now also Z101.1
- net LED16: no longer Z101.1
- net MATRIX_CS: now also T0.1; no longer Q1.1
- net MISO: now also EEP.2; no longer U5.2
- net MOSI: now also EEP.5; no longer U5.5
- net N$116: now also SW_NEN.2@1, SW_NEN.2@2; no longer SW_NEN.1@1, SW_NEN.1@2
- net N$117: now also SW_NP.2@1, SW_NP.2@2; no longer SW_NP.1@1, SW_NP.1@2
- net N$54: now also T0.2; no longer Q1.2
- net RED10: no longer Z103.3
- net RED8: now also Z102.3
- net RED9: now also Z103.3; no longer Z102.3
- net ROW0: now also T2.2, T3.2; no longer FET1.2, FET2.2
- net ROW2: now also SW_NP.1@1, SW_NP.1@2; no longer SW_NP.2@1, SW_NP.2@2
- net ROW4: now also SW_NEN.1@1, SW_NEN.1@2; no longer SW_NEN.2@1, SW_NEN.2@2
- net S13: now also T2.3; no longer FET1.3
- net S17: now also T3.3; no longer FET2.3
- net SCK: now also EEP.6; no longer U5.6
- net VCC_1: now also C20.1, M_M2.5; no longer C23.1
- net VCC_2: now also C23.1, EEP.3, EEP.7, EEP.8, LM1117.4, RST.1, S1.1, S1.2; no longer C20.1, Q2.2, R67.2, R69.2, U5.3, U5.7, U5.8
Routing:
- net VCC_2: track 0.00 -> 1299.3 mm, vias 0 -> 36
- net ROW0: track 0.00 -> 437.9 mm, vias 0 -> 4
- net ROW1: track 0.00 -> 396.1 mm, vias 0 -> 1
- net ROW2: track 0.00 -> 391.8 mm, vias 0 -> 3
- net ROW4: track 0.00 -> 366.9 mm, vias 0 -> 2
- net ROW3: track 0.00 -> 354.8 mm, vias 0 -> 3
- net USB_D_N: track 0.00 -> 286.1 mm, vias 0 -> 2
- net USB_D_P: track 0.00 -> 285.6 mm, vias 0 -> 2
- net VCC_1: track 0.00 -> 270.9 mm, vias 0 -> 6
- net ROW5: track 0.00 -> 270.2 mm, vias 0 -> 1
- net BOOT0: track 0.00 -> 196.9 mm, vias 0 -> 1
- net ENC_B: track 0.00 -> 194.8 mm, vias 0 -> 6
- net !RESET: track 0.00 -> 191.6 mm, vias 0 -> 1
- net ENC_A: track 0.00 -> 180.6 mm, vias 0 -> 5
- net COL11: track 0.00 -> 174.7 mm, vias 0 -> 7
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
Commit message: .
Parts:
- removed J_5V: 5V SRC SELECT, SparkFun-Jumpers:SMT-JUMPER_3_1-NC_TRACE_SILK
- removed T0: 2N7002, adafruit:SOT23
- removed T1: DTC123JKAT146, __temp_to_delete:TRANS_DTA113TKAT_ROM
- added 5V: (no value), SparkFun-Connectors:1X02
- added C33: 1uF, rcl:C0603
- added Q0, Q1, Q2: 2N7002, ts_custom_nick_nacks:SOT23-3
- added R23, R27: 10K, rcl:R0603
- added R24: 100K, rcl:R0603
- added R25: 100R, rcl:R0603
- added R26: 1K, rcl:R0603
- added U$1, U$2, U$3: FIDUCIAL, __temp_to_delete:FIDUCIAL
- D100: value (none) -> 1N4148
- R20: value 100R -> 330K
- R21: value 330K -> 1M
- R22: value 1M -> 10K
- moved U6 167.0 mm to (12.0, 62.0)
- moved R71 164.5 mm to (7.75, 63.0), turned to 180 degrees
- moved D102 137.7 mm to (26.2, 10.4)
- moved R15 107.6 mm to (238.5, 35.0), turned to 270 degrees
- moved R11 104.7 mm to (235.0, 35.0), turned to 270 degrees
- moved JKEY 102.3 mm to (38.0, 33.3)
- moved R13 101.6 mm to (21.0, 44.0), turned to 270 degrees
- moved D101 98.1 mm to (34.2, 48.5)
- moved R8 95.5 mm to (24.5, 44.0), turned to 270 degrees
- moved R7 92.7 mm to (28.0, 44.0), turned to 270 degrees
- moved C6 91.9 mm to (245.0, 42.0), turned to 270 degrees
- moved C7 88.2 mm to (247.1, 42.0), turned to 270 degrees
- moved C1 86.3 mm to (29.7, 49.2), turned to 90 degrees
- moved C8 85.0 mm to (239.0, 49.0)
- moved C9 83.4 mm to (239.0, 47.0)
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Connections:
- net N$149 renamed U3_TO_U4
- net N$162 renamed U2_TO_U3
- removed net GND2: R0.1, R0.2, R0.3, R0.4, R1.1, R1.2, R1.3, R1.4, R2.1, R2.2, R2.3, R2.4, R3.1, R3.2, R3.3, R3.4, R4.1, R4.2, R4.3, R4.4, R5.1, R5.2, R5.3, R5.4
- removed net LOAD_SWITCH_OUT: J_5V.1, U6.5
- removed net N$54: T0.2
- new net N$12: Q1.1, R26.1, R27.1
- new net N$13: D100.A, R26.2, RST.2, S1.3, S1.4
- new net N$5: D100.C, R20.2
- new net PB5: JPWM.4, U1.41
- net !RESET: now also C30.2, R25.2; no longer C30.1, R20.2
- net BLU3: now also R7.6; no longer R7.8
- net BLU4: now also R7.8; no longer R7.6
- net BOOT0: now also R20.1, R21.2, R22.2; no longer R21.1, R22.1
- net GND: now also 5V.2, C30.1, C33.1, Q0.2, Q1.2, Q2.2, R0.1, R0.2, R0.3, R0.4, R1.1, R1.2, R1.3, R1.4, R2.1, R2.2, R2.3, R2.4, R21.1, R24.2, R27.2, R3.1, R3.2, R3.3, R3.4, R4.1, R4.2, R4.3, R4.4, R5.1, R5.2, R5.3, R5.4; no longer C30.2, JTAG.7, R22.2, T1.3
- net GRN3: now also R7.5; no longer R7.7
- net GRN4: now also R7.7; no longer R7.5
- net LATCH: now also Q0.3; no longer T0.3
- net MATRIX_CS: now also Q0.1; no longer T0.1
- net N$11: now also Q1.3, R23.2, R25.1; no longer D100.A, RST.2, S1.3, S1.4, T1.2
- net N$7: now also Q2.3, R22.1; no longer R20.1, T1.1
- net N$9: now also Q2.1, R23.1, R24.1; no longer D100.C, R21.2
- net PA8: now also JPWM.3; no longer JPWM.4
- net RED4: now also R13.7; no longer R13.8
- net RED5: now also R13.6; no longer R13.7
- net RED6: now also R13.5; no longer R13.6
- net VCC_1: now also 5V.1, C33.2; no longer JPWM.1, J_5V.3
- net VCC_2: now also JPWM.1; no longer JPWM.2
- net VCC_LED: now also U6.5; no longer J_5V.2
- net WKUP: now also JPWM.2; no longer JPWM.3
- net XB3: now also R7.3; no longer R7.1
- net XB4: now also R7.1; no longer R7.3
- net XG3: now also R7.4; no longer R7.2
- net XG4: now also R7.2; no longer R7.4
- net XR4: now also R13.2; no longer R13.1
- net XR5: now also R13.3; no longer R13.2
- net XR6: now also R13.4; no longer R13.3
Routing:
- net MISO: track 53.4 -> 431.7 mm, vias 3 -> 9
- net SCK: track 49.5 -> 423.3 mm, vias 3 -> 12
- net GRN1: track 0.00 -> 363.2 mm, vias 0 -> 14
- net BLU1: track 0.00 -> 346.1 mm, vias 0 -> 12
- net RED1: track 0.00 -> 344.3 mm, vias 0 -> 14
- net RED6: track 0.00 -> 341.0 mm, vias 0 -> 8
- net GRN6: track 0.00 -> 336.9 mm, vias 0 -> 10
- net BLU6: track 0.00 -> 311.6 mm, vias 0 -> 10
- net LED8: track 0.00 -> 285.9 mm, vias 0 -> 13
- net LED6: track 0.00 -> 276.4 mm, vias 0 -> 11
- net LED9: track 0.00 -> 264.9 mm, vias 0 -> 7
- net GRN2: track 0.00 -> 263.3 mm, vias 0 -> 11
- net GRN3: track 0.00 -> 256.5 mm, vias 0 -> 12
- net LED7: track 0.00 -> 255.5 mm, vias 0 -> 14
- net MATRIX_CS: track 77.1 -> 328.7 mm, vias 2 -> 8
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Other:
- board text removed: "DIP SW"

Commit message: .
Parts:
- removed H_RS: MX-STABS-200U, ts_keyboards:MX-STABS-200U
- added C34: 1uF, rcl:C0603
- added G1, G2, G3, G4, G5, G6: MGEEK-M2-HOLE, untitled:MGEEK-M2-HOLE
- added H1, H10, H11, H12, H2, H3, H4, H5, H6, H7, H8, H9: BRURAL-1800-HOLE, untitled:BRUTAL-1800-HOLE
- added LOGO1: OSHW-LOGOL, random_logos:OSHW-LOGO-L
- added R72: 1K, rcl:R0603
- added U$4: QMK_LOGO, random_logos:QMK_LOGO
- added U$5, U$6: TECSMITH-LOGOLONG, random_logos:TECSMITH-NAME
- added U5: TPS22995H-Q1, __untitled:SOT-23-THIN-6_DDC_TEX
- Z1, Z10, Z101, Z102, Z103, Z104, Z105, Z106, Z107, Z11, Z12, Z13, Z14, Z15, Z16, Z17, Z18, Z2, Z20, Z21, Z22, Z23, Z24, Z25, Z26, Z27, Z28, Z29, Z3, Z30, Z31, Z32, Z33, Z34, Z35, Z36, Z37, Z38, Z39, Z4, Z40, Z41, Z42, Z43, Z44, Z45, Z46, Z47, Z48, Z49, Z5, Z50, Z51, Z52, Z53, Z54, Z55, Z56, Z57, Z58, Z59, Z6, Z60, Z61, Z62, Z63, Z64, Z65, Z66, Z67, Z68, Z69, Z7, Z70, Z71, Z72, Z73, Z74, Z75, Z76, Z77, Z78, Z79, Z8, Z80, Z81, Z82, Z83, Z84, Z85, Z86, Z87, Z88, Z89, Z9, Z90, Z91, Z92, Z93, Z94, Z95, Z96, Z97, Z98, Z99: value 156120M173000 -> 156120M173000MILL; device ts_keyboards:156120M173000 -> ts_keyboards:156120M173000-MILL
- Z19: device ts_keyboards:156120M173000 -> ts_keyboards:156120M173000-MILL
- moved U6 250.6 mm to (261.5, 38.5), turned to 90 degrees
- moved C6 12.6 mm to (255.0, 49.7), turned to 0 degrees
- moved C7 9.72 mm to (255.0, 47.6), turned to 0 degrees
- moved D107 9.53 mm to (159.5, 14.3), turned to 180 degrees
- moved R70 9.53 mm to (159.5, 14.3), turned to 180 degrees
- moved JI2C 7.62 mm to (249.8, 15.6), flipped to the bottom, turned to 270 degrees
- moved R11 5.22 mm to (233.5, 40.0)
- moved R15 5.22 mm to (237.0, 40.0)
- moved D102 5.05 mm to (21.2, 10.3)
- moved T3 3.28 mm to (349.1, 109.5)
- moved D99 1.11 mm to (337.5, 10.3)
- moved C10 1.00 mm to (235.0, 64.0)
- moved R39 1.00 mm to (237.1, 64.0)
- moved R40 1.00 mm to (239.1, 64.0)
- moved D89 0.91 mm to (30.1, 10.3)
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Connections:
- removed net LED_SBD: C10.2, C5.2, R37.2, R39.2, U_LED1.26, U_LED2.26
- removed net VCC_LED: C1.2, C2.2, C3.2, C4.2, C6.2, C7.2, C8.2, C9.2, U6.5, U_LED1.22, U_LED1.5, U_LED2.22, U_LED2.5
- new net N$1: R72.2, U6.6
- new net VCC_LED_1: C1.2, C2.2, C3.2, C4.2, U5.5, U_LED1.22, U_LED1.5
- new net VCC_LED_2: C6.2, C7.2, C8.2, C9.2, U6.5, U_LED2.22, U_LED2.5
- net GND: now also C34.1, R72.1, U5.4
- net LED_PWR_EN: now also C10.2, C5.2, R37.2, R39.2, U5.3, U_LED1.26, U_LED2.26
- net N$135: now also U5.6; no longer U6.6
- net VCC_1: now also C34.2, U5.1, U5.2
Routing:
- net LED_PWR_EN: track 4.11 -> 350.1 mm, vias 1 -> 11
- net LED1_CS: track 92.5 -> 349.2 mm, vias 3 -> 10
- net SYNC: track 35.7 -> 277.1 mm, vias 1 -> 4
- net MOSI: track 281.0 -> 429.3 mm, vias 3 -> 10
- net VCC_1: track 404.5 -> 546.2 mm, vias 7 -> 10
- net ROW5: track 380.3 -> 457.3 mm, vias 11 -> 13
- net VCC_LED_1: track 0.00 -> 75.9 mm, vias 0 -> 2
- net VCC_LED: track 75.9 -> 0.00 mm, vias 2 -> 0
- net LED2_CS: track 29.2 -> 101.2 mm, vias 1 -> 4
- net MISO: track 431.7 -> 502.7 mm, vias 9 -> 11
- net SCK: track 423.3 -> 487.5 mm, vias 12 -> 16
- net VCC_LED_2: track 0.00 -> 52.2 mm, vias 0 -> 3
- net GND: track 33.9 -> 61.4 mm, vias 44 -> 39
- net TECSMITH: track 0.00 -> 25.0 mm
- net XR9: track 0.00 -> 24.4 mm, vias 0 -> 2
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Other:
- board text added: "'"
- board text added: "(c) 2024 Vino Rodrigues https://c1k.it/vr99"
- board text added: "*"
- board text added: "+"
- board text added: ","
- board text added: "-"
- board text added: "."
- board text added: "/"
- board text added: "0"
- board text added: "1"
- board text added: "2"
- board text added: "2024 Vino Rodrigues"
- board text added: "3"
- board text added: "3V3"
- board text added: "4"
- board text added: "5"
- board text added: "6"
- board text added: "7"
- board text added: "8"
- board text added: "9"
- board text added: ";"
- board text added: "A"
- board text added: "B"
- board text added: "Bsp"
- board text added: "C"
- board text added: "CS"
- board text added: "Cps"
- board text added: "Ctl"
- board text added: "D"
- board text added: "DC"
- board text added: "E"
- board text added: "Ent"
- board text added: "Esc"
- board text added: "F"
- board text added: "F1"
- board text added: "F10"
- board text added: "F11"
- board text added: "F12"
- board text added: "F2"
- board text added: "F3"
- board text added: "F4"
- board text added: "F5"
- board text added: "F6"
- board text added: "F7"
- board text added: "F8"
- board text added: "F9"
- board text added: "G"
- board text added: "GND"
- board text added: "H"
- board text added: "I"
- board text added: "J"
- board text added: "K"
- board text added: "L"
- board text added: "M"
- board text added: "MISO"
- board text added: "MOSI"
- board text added: "N"
- board text added: "Num"
- board text added: "O"
- board text added: "Open Hardware"
- board text added: "P"
- board text added: "PA0"
- board text added: "PA8"
- board text added: "PB5"
- board text added: "Q"
- board text added: "R"
- board text added: "RESET"
- board text added: "Rev A"
- board text added: "S"
- board text added: "SCK"
- board text added: "SCL"
- board text added: "SDA"
- board text added: "Sft"
- board text added: "Spc"
- board text added: "T"
- board text added: "Tab"
- board text added: "U"
- board text added: "V"
- board text added: "VR99"
- board text added: "VR99 Keyboard"
- board text added: "W"
- board text added: "X"
- board text added: "Y"
- board text added: "Z"
- board text added: "["
- board text added: "\\"
- board text added: "]"
- board text added: "c"
- board text added: "~"
