File: EAGLE/vr99/vr99-south-revA.sch (EAGLE design)
At the start: 405 parts, among them Q1 2N7002, Q2 DMG2305UX-7, U1 STM32F411CEU7THERM, U2 74HC589A_DT, U3 74HC589A_DT, U4 74HC589A_DT, U5 M25C, U6 TPS22995H-Q1, Y1 32.768kHz ±20ppm 6pF, Y2 25MHz 9pF

Commit message: .
Parts:
- added C31, C32: 100nF, rcl:C-EUC0603
- added FET1, FET2: AO3401A, __untitled:AO3401A
- added R0, R19: 10K, rcl:R-EU_R0603
- R18: value 5.1K -> 10K
Connections:
- removed net ENC_S: R18.2, SW_F13G$1.S, SW_F17G$1.S, U1A.PA8
- removed net N$144: D101.A, JKEY.3
- removed net N$38: D14.A, SW_F13G$2.P
- removed net ROW6: SW_A.S, SW_CL.S, SW_CS.S, SW_D.S, SW_ENT.S, SW_F.S, SW_G.S, SW_H.S, SW_J.S, SW_K.S, SW_L.S, SW_N4.S, SW_N5.S, SW_N6.S, SW_QU.S, SW_S.S
- new net COL_G1: R5.5, U2.A
- new net COL_G2: R0.2, U4.A, U4.F, U4.G, U4.H
- new net N$3: FET1.G, R18.1, SW_F13G$1.S
- new net N$5: FET2.G, R19.1, SW_F17G$1.S
- new net S13: D14.A, FET1.D, SW_F13G$2.P
- new net S17: D18.A, FET2.D, SW_F17G$2.P
- net ENC_A: now also C31.1
- net ENC_B: now also C32.1, R17.1; no longer R17.2
- net GND: now also C31.2, C32.2; no longer U2.A, U4.A, U4.F, U4.G, U4.H
- net GND2: now also R0.1, R5.4
- net N$4: now also D101.A, JKEY.4; no longer D18.A, SW_F17G$2.P
- net ROW0: now also FET1.S, FET2.S
- net ROW3: now also JKEY.2, SW_A.S, SW_CL.S, SW_CS.S, SW_D.S, SW_ENT.S, SW_F.S, SW_G.S, SW_H.S, SW_J.S, SW_K.S, SW_L.S, SW_N4.S, SW_N5.S, SW_N6.S, SW_QU.S, SW_S.S
- net ROW5: now also JKEY.3; no longer JKEY.2, JKEY.4
- net VCC_2: now also R17.2, R18.2, R19.2; no longer R17.1, R18.1
Other:
- moved on the sheet: D101, R16, R17, R18, SW_F13G$1, SW_F17G$1

Commit message: .
Parts:
- removed D201, D202: 1N4148, adafruit:DIODESOT23_REFLOW
- removed FET1, FET2: AO3401A, __untitled:AO3401A
- removed J1: (no value), SparkFun-Connectors:CONN_02
- removed Q2: DMG2305UX-7, SparkFun-DiscreteSemi:MOSFET_PCH-DMG2305UX-7
- removed R67, R68: 100K, rcl:R-EU_R0603
- removed R69: /DNP/, rcl:R-EU_R0603
- removed U5: M25C, ts_kb_mcu:M25C
- added D100: (no value), jlcpcb_basic_parts:1N5819WS
- added EEP: M25C, ts_kb_mcu:M25C
- added M_M2: SM05B-SRSS-TB(LF)(SN), __temp_to_delete:SM05B-SRSS-TB(LF)(SN)
- added R20: 100R, rcl:R-EU_R0603
- added R21: 330K, rcl:R-EU_R0603
- added R22: 1M, rcl:R-EU_R0603
- added RST: (no value), SparkFun-Connectors:CONN_02
- added T1: DTC123JKAT146, __temp_to_delete:DTC123JKAT146
- added T2, T3: AO3401A, __untitled:AO3401A
- C20: value 100nF -> 22uF; device SparkFun-Capacitors:0.1UF-0603-25V-5% -> SparkFun-Capacitors:0.22UF-0603-25V-10%
- C22: value 22uF -> 100nF; device SparkFun-Capacitors:0.22UF-0603-25V-10% -> SparkFun-Capacitors:0.1UF-0603-25V-5%
- C29: value (none) -> 10uF; device rcl:C-EUC0603 -> rcl:C-EUC0805
- JPWM: device SparkFun-Connectors:CONN_04 -> SparkFun-Connectors:CONN_05NO_SILK
- JTAG: value DNP -> CORTEX_JTAG_DEBUG_PTH_NS; device SparkFun-Connectors:CONN_05X2NO_SILK -> SparkFun-Connectors:CORTEX_JTAG_DEBUG_PTH_NS
- R0: device rcl:R-EU_R0603 -> ts_keyboards:R-EU-4
- Y2: device SparkFun-Clocks:CRYSTAL-24MHZ" -> __temp_to_delete:CRYSTAL2.5X2.0
- renumbered Q1 to T0
Connections:
- net N$140 renamed USB_N
- net N$141 renamed USB_P
- removed net !BOOT: C30.1, D202.A, Q2.G, R67.1
- removed net COL_G1: R5.5, U2.A
- removed net COL_G2: R0.2, U4.A, U4.F, U4.G, U4.H
- removed net LED_SDB: U1A.PB5
- removed net N$3: FET1.G, R18.1, SW_F13G$1.S
- removed net N$5: FET2.G, R19.1, SW_F17G$1.S
- removed net RESET: D201.C, D202.C, J1.2, S1.2
- removed net USB_DN: R45.1, UDB1.DN, UDB2.DN
- removed net USB_DP: R46.1, UDB1.DP, UDB2.DP
- new net G1: R4.8, U2.A
- new net G2: R2.8, U3.A
- new net G3: R1.8, U4.A
- new net G4: R0.7, U4.F
- new net G5: R0.6, U4.G
- new net G6: R0.5, U4.H
- new net N$11: D100.A, RST.2, S1.2, T1.1
- new net N$6: R19.1, SW_F17G$1.S, T3.G
- new net N$7: R20.1, T1.2
- new net N$8: R18.1, SW_F13G$1.S, T2.G
- new net N$9: D100.C, R21.2
- new net PA8: JPWM.4, U1A.PA8
- new net USB_D_N: M_M2.P$3, R45.1, UDB1.DN, UDB2.DN
- new net USB_D_P: M_M2.P$4, R46.1, UDB1.DP, UDB2.DP
- net !RESET: now also C30.1, R20.2; no longer C29.2, D201.A, R69.1
- net BLU10: no longer Z103.B
- net BLU8: now also Z102.B
- net BLU9: now also Z103.B; no longer Z102.B
- net BOOT0: now also C29.1, R21.1, R22.1; no longer Q2.D, R68.1
- net COL0: now also R4.7; no longer R4.8
- net COL1: now also R4.6; no longer R4.7
- net COL10: now also R3.8; no longer R2.5
- net COL11: now also R3.7; no longer R3.8
- net COL12: now also R3.6; no longer R3.7
- net COL13: now also R3.5; no longer R3.6
- net COL14: now also R1.7; no longer R1.8
- net COL15: now also R1.6; no longer R1.7
- net COL16: now also R1.5; no longer R1.6
- net COL17: now also R0.8; no longer R1.5
- net COL2: now also R4.5; no longer R4.6
- net COL3: now also R5.8; no longer R4.5
- net COL4: now also R5.7; no longer R5.8
- net COL5: now also R5.6; no longer R5.7
- net COL6: now also R5.5; no longer R5.6
- net COL7: now also R2.7; no longer R2.8
- net COL8: now also R2.6; no longer R2.7
- net COL9: now also R2.5; no longer R2.6
- net EE_CS: now also EEP.!CS; no longer U5.!CS
- net GND: now also C29.2, EEP.GND, JPWM.5, JTAG.GND@3, JTAG.GND@5, JTAG.GNDDTCT, JTAG.KEY, M_M2.P$1, M_M2.P$2, M_M2.P$6, R22.2, T1.3, Y2.2, Y2.4; no longer C29.1, J1.1, JPWM.4, JTAG.3, JTAG.5, JTAG.9, R68.2, S1.1, U3.A, U5.GND
- net GND2: now also R0.2, R0.3, R0.4, R3.4
- net GRN10: no longer Z103.G
- net GRN8: now also Z102.G
- net GRN9: now also Z103.G; no longer Z102.G
- net J_RST: now also JTAG.!RESET; no longer JTAG.10
- net J_TCK: now also JTAG.SWDCLK/TCK; no longer JTAG.4
- net J_TDI: now also JTAG.NC/TDI; no longer JTAG.8
- net J_TDO: now also JTAG.SWO/TDO; no longer JTAG.6
- net J_TMS: now also JTAG.SWDIO/TMS; no longer JTAG.2
- net LED15: now also Z101.A
- net LED16: no longer Z101.A
- net MISO: now also EEP.DO; no longer U5.DO
- net MOSI: now also EEP.DIO; no longer U5.DIO
- net N$116: now also SW_NEN.S; no longer SW_NEN.P
- net N$117: now also SW_NP.S; no longer SW_NP.P
- net RED10: no longer Z103.R
- net RED8: now also Z102.R
- net RED9: now also Z103.R; no longer Z102.R
- net ROW0: now also T2.S, T3.S; no longer FET1.S, FET2.S
- net ROW2: now also SW_NP.P; no longer SW_NP.S
- net ROW4: now also SW_NEN.P; no longer SW_NEN.S
- net S13: now also T2.D; no longer FET1.D
- net S17: now also T3.D; no longer FET2.D
- net SCK: now also EEP.CLK; no longer U5.CLK
- net VCC_1: now also C20.1, M_M2.P$5; no longer C23.1
- net VCC_2: now also C23.1, EEP.!HLD, EEP.!WP, EEP.VCC, JTAG.VCC, LM1117.OUT@1, RST.1, S1.1; no longer C20.1, JTAG.1, Q2.S, R67.2, R69.2, U5.!HLD, U5.!WP, U5.VCC
- net Y2I: now also Y2.3; no longer Y2.2
Other:
- note added: "Debug Header"
- note added: "Hard Reset"
- note added: "Monsgeek M2 Drop-In Mounting Holes (marked with Triangle) and KST connector pinout need to be confirmed still."
- note added: "Optional / Aux SPI break-out"
- note added: "Optional I2C break-out"
- note added: "Optional PWM break-out"
- note added: "SKYLONG Rotary Encoder 2 Positions - Only use 1"
- note added: "Shift/Reg / Col-scan Pulldowns"
- note added: "Shift/Reg Decoupling"
- note removed: "!RESET"
- note removed: "BOOT0 Inversion"
- note removed: "COL-SCAN PULL-DOWNS"
- moved on the sheet: C19, C20, C22, C23, C28, C30, D101, D102, D107, JI2C, JKEY, JSPI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

Commit message: .
Parts:
- removed J_5V: 5V SRC SELECT, SparkFun-Jumpers:JUMPER-SMT_3_1-NC_TRACE_SILK
- removed T0: 2N7002, adafruit:MOSFET-NREFLOW
- removed T1: DTC123JKAT146, __temp_to_delete:DTC123JKAT146
- added 5V: (no value), SparkFun-Connectors:CONN_02
- added C33: 1uF, rcl:C-EUC0603
- added Q0, Q1, Q2: 2N7002, ts_custom_nick_nacks:2N7002-BSS138
- added R23, R27: 10K, rcl:R-EU_R0603
- added R24: 100K, rcl:R-EU_R0603
- added R25: 100R, rcl:R-EU_R0603
- added R26: 1K, rcl:R-EU_R0603
- added U$1, U$2, U$3: FIDUCIAL, __temp_to_delete:FIDUCIAL
- D100: value (none) -> 1N4148
- R20: value 100R -> 330K
- R21: value 330K -> 1M
- R22: value 1M -> 10K
Connections:
- net N$149 renamed U3_TO_U4
- net N$162 renamed U2_TO_U3
- removed net GND2: R0.1, R0.2, R0.3, R0.4, R1.1, R1.2, R1.3, R1.4, R2.1, R2.2, R2.3, R2.4, R3.1, R3.2, R3.3, R3.4, R4.1, R4.2, R4.3, R4.4, R5.1, R5.2, R5.3, R5.4
- removed net LOAD_SWITCH_OUT: J_5V.1, U6.OUT
- removed net N$54: T0.S
- new net N$12: Q1.G, R26.1, R27.1
- new net N$13: D100.A, R26.2, RST.2, S1.2
- new net N$5: D100.C, R20.2
- new net PB5: JPWM.4, U1A.PB5
- net !RESET: now also C30.2, R25.2; no longer C30.1, R20.2
- net BLU3: now also R7.6; no longer R7.8
- net BLU4: now also R7.8; no longer R7.6
- net BOOT0: now also R20.1, R21.2, R22.2; no longer R21.1, R22.1
- net GND: now also 5V.2, C30.1, C33.1, Q0.S, Q1.S, Q2.S, R0.1, R0.2, R0.3, R0.4, R1.1, R1.2, R1.3, R1.4, R2.1, R2.2, R2.3, R2.4, R21.1, R24.2, R27.2, R3.1, R3.2, R3.3, R3.4, R4.1, R4.2, R4.3, R4.4, R5.1, R5.2, R5.3, R5.4; no longer C30.2, JTAG.KEY, R22.2, T1.3
- net GRN3: now also R7.5; no longer R7.7
- net GRN4: now also R7.7; no longer R7.5
- net LATCH: now also Q0.D; no longer T0.D
- net MATRIX_CS: now also Q0.G; no longer T0.G
- net N$11: now also Q1.D, R23.2, R25.1; no longer D100.A, RST.2, S1.2, T1.1
- net N$7: now also Q2.D, R22.1; no longer R20.1, T1.2
- net N$9: now also Q2.G, R23.1, R24.1; no longer D100.C, R21.2
- net PA8: now also JPWM.3; no longer JPWM.4
- net RED4: now also R13.7; no longer R13.8
- net RED5: now also R13.6; no longer R13.7
- net RED6: now also R13.5; no longer R13.6
- net VCC_1: now also 5V.1, C33.2; no longer JPWM.1, J_5V.3
- net VCC_2: now also JPWM.1; no longer JPWM.2
- net VCC_LED: now also U6.OUT; no longer J_5V.2
- net WKUP: now also JPWM.2; no longer JPWM.3
- net XB3: now also R7.3; no longer R7.1
- net XB4: now also R7.1; no longer R7.3
- net XG3: now also R7.4; no longer R7.2
- net XG4: now also R7.2; no longer R7.4
- net XR4: now also R13.2; no longer R13.1
- net XR5: now also R13.3; no longer R13.2
- net XR6: now also R13.4; no longer R13.3
Other:
- note added: "(c) Gondolindrim - Figure 28 from https://acheronproject.com/reset_article_1/reset_article_1/"
- note added: "5V Test Pad"
- note added: "LED POWER SWITCH /w optional direct pwr"
- note added: "Monsgeek M2 Drop-In Mounting Holes (marked with Triangle) and JST connector pinout need to be confirmed still."
- note added: "NOTE (to self) There is no driver for the IS31FL3743B SPI Also remember that each IC needs it's own CS pin. This will make the driver a tad more challanging to write. Good luck. ..or.. Replace this with the IS31FL3743A I2C variant."
- note added: "RT = 1K for 166us slew rate on a 5V supply"
- note removed: "LED POWER SWITCH /DNP/ (Optional)"
- note removed: "Monsgeek M2 Drop-In Mounting Holes (marked with Triangle) and KST connector pinout need to be confirmed still."
- note removed: "NOTE There is no driver for the IS31FL3743B SPI Also remember that each IC needs it's own CS pin. This will make the driver a tad more challanging to write. Good luck. ..or.. Replace this with the IS31FL3743A I2C variant."
- moved on the sheet: C29, C3, C30, C4, C8, C9, D100, R20, R21, R22, R65, RST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

Commit message: .
Parts:
- removed H_RS: MX-STABS-200U, ts_keyboards:MX-STABS-200U
- added C34: 1uF, rcl:C-EUC0603
- added G1, G2, G3, G4, G5, G6: MGEEK-M2-HOLE, untitled:MGEEK-M2-HOLE
- added H1, H10, H11, H12, H2, H3, H4, H5, H6, H7, H8, H9: BRURAL-1800-HOLE, untitled:BRURAL-1800-HOLE
- added LOGO1: OSHW-LOGOL, random_logos:OSHW-LOGOL
- added R72: 1K, rcl:R-EU_R0603
- added U$4: QMK_LOGO, random_logos:QMK_LOGO
- added U$5: TECSMITH-LOGOLONG, random_logos:TECSMITH-LOGOLONG
- added U5: TPS22995H-Q1, __untitled:TPS22995H-Q1
- Z1, Z10, Z101, Z102, Z103, Z104, Z105, Z106, Z107, Z11, Z12, Z13, Z14, Z15, Z16, Z17, Z18, Z2, Z20, Z21, Z22, Z23, Z24, Z25, Z26, Z27, Z28, Z29, Z3, Z30, Z31, Z32, Z33, Z34, Z35, Z36, Z37, Z38, Z39, Z4, Z40, Z41, Z42, Z43, Z44, Z45, Z46, Z47, Z48, Z49, Z5, Z50, Z51, Z52, Z53, Z54, Z55, Z56, Z57, Z58, Z59, Z6, Z60, Z61, Z62, Z63, Z64, Z65, Z66, Z67, Z68, Z69, Z7, Z70, Z71, Z72, Z73, Z74, Z75, Z76, Z77, Z78, Z79, Z8, Z80, Z81, Z82, Z83, Z84, Z85, Z86, Z87, Z88, Z89, Z9, Z90, Z91, Z92, Z93, Z94, Z95, Z96, Z97, Z98, Z99: value 156120M173000 -> 156120M173000MILL; device ts_keyboards:156120M173000 -> ts_keyboards:156120M173000MILL
- Z19: device ts_keyboards:156120M173000 -> ts_keyboards:156120M173000MILL
Connections:
- removed net LED_SBD: C10.2, C5.2, R37.2, R39.2, U_LED1.SDB, U_LED2.SDB
- removed net VCC_LED: C1.2, C2.2, C3.2, C4.2, C6.2, C7.2, C8.2, C9.2, U6.OUT, U_LED1.PVCC, U_LED1.VCC, U_LED2.PVCC, U_LED2.VCC
- new net N$1: R72.2, U6.RT
- new net VCC_LED_1: C1.2, C2.2, C3.2, C4.2, U5.OUT, U_LED1.PVCC, U_LED1.VCC
- new net VCC_LED_2: C6.2, C7.2, C8.2, C9.2, U6.OUT, U_LED2.PVCC, U_LED2.VCC
- net GND: now also C34.1, R72.1, U5.G
- net LED_PWR_EN: now also C10.2, C5.2, R37.2, R39.2, U5.ON, U_LED1.SDB, U_LED2.SDB
- net N$135: now also U5.RT; no longer U6.RT
- net VCC_1: now also C34.2, U5.BI, U5.IN
Other:
- note added: "LED POWER SWITCH"
- note removed: "LED POWER SWITCH /w optional direct pwr"
- moved on the sheet: C33, R71, U6
