File: EAGLE/vr99/vr99-revA.brd (EAGLE design)
At the start: 369.5 x 121.8 mm, 445 parts, among them Q0 2N7002, Q1 2N7002, Q2 2N7002, T2 AO3401A, T3 AO3401A, U1 STM32F411CEU7THERM, U2 74HC589A_DT, U3 74HC589A_DT, U4 74HC589A_DT, U5 TPS22995H-Q1, U6 TPS22995H-Q1, Y1 32.768kHz ±20ppm 6pF, Y2 25MHz 9pF

Commit message: pre- GND routing save
Parts:
- removed D101, D102: DNP, jlcpcb_basic_parts:SOD-123
- removed JKEY: MOLEX_0781710005, molex-pico-ezmate:MOLEX_781710005
- added JDIP: MOLEX_0781710006, molex-pico-ezmate:MOLEX_781710006
- D107: device SparkFun-LED:LED-0603 -> untitled:LED-RM-MILL
- JTAG: value CORTEX_JTAG_DEBUG_PTH_NS -> TC2050IDC-NL; device SparkFun-Connectors:2X5-PTH-1.27MM-NO_SILK -> ts_custom_nick_nacks:TC2050-IDC-NL
- moved U$5 10.8 mm to (175.5, 20.8)
- moved R41 7.09 mm to (256.9, 22.0), turned to 90 degrees
- moved JTAG 5.00 mm to (285.0, 89.0)
- moved R42 4.12 mm to (254.0, 22.0), turned to 90 degrees
- moved R27 3.72 mm to (88.6, 11.7), turned to 0 degrees
- moved R70 3.00 mm to (159.5, 17.3)
- moved U$4 2.61 mm to (87.6, 60.1)
- moved C10 1.79 mm to (236.8, 63.8)
- moved R39 1.76 mm to (238.8, 63.8)
- moved R40 1.74 mm to (240.8, 63.8)
- moved C7 1.25 mm to (255.5, 48.8)
- moved C6 1.23 mm to (255.5, 50.8)
- moved R45 1.20 mm to (282.0, 74.8)
- moved R46 1.20 mm to (284.1, 74.8)
- moved R10 1.00 mm to (253.0, 66.0)
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Connections:
- removed net N$156: D102.A, JKEY.5
- removed net N$4: D101.A, JKEY.4
- new net N$10: JDIP.NC1, JDIP.NC2
- net COL3: now also JDIP.3
- net COL4: now also JDIP.4; no longer D101.C
- net COL6: now also JDIP.5; no longer D102.C
- net COL7: now also JDIP.6
- net GND: now also JDIP.1, R12.4, R12.5, R13.1, R13.8, R14.4, R14.5, R15.1, R15.8; no longer JKEY.1, JKEY.NC1, JKEY.NC2
- net J_TCK: now also JTAG.2; no longer JTAG.4
- net J_TMS: now also JTAG.4; no longer JTAG.2
- net RED10: now also R15.5; no longer R15.8
- net ROW3: no longer JKEY.2
- net ROW5: now also JDIP.2; no longer JKEY.3
- net XR10: now also R15.4; no longer R15.1
Routing:
- net RED12: track 0.00 -> 336.7 mm, vias 0 -> 24
- net BLU12: track 0.00 -> 328.7 mm, vias 0 -> 14
- net GRN12: track 0.00 -> 327.0 mm, vias 0 -> 26
- net GRN9: track 0.00 -> 315.2 mm, vias 0 -> 18
- net LED14: track 1.31 -> 306.4 mm, vias 1 -> 17
- net RED9: track 0.00 -> 297.6 mm, vias 0 -> 18
- net GRN8: track 0.00 -> 274.5 mm, vias 0 -> 16
- net GRN7: track 0.00 -> 274.2 mm, vias 0 -> 14
- net LED16: track 0.00 -> 271.8 mm, vias 0 -> 17
- net BLU9: track 3.93 -> 275.3 mm, vias 1 -> 17
- net BLU7: track 0.00 -> 265.0 mm, vias 0 -> 13
- net LED20: track 0.00 -> 263.4 mm, vias 0 -> 13
- net LED19: track 0.00 -> 263.2 mm, vias 0 -> 10
- net GRN11: track 0.00 -> 263.1 mm, vias 0 -> 10
- net GRN10: track 0.00 -> 262.2 mm, vias 0 -> 12
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Other:
- board text removed: "c"

Commit message: post GND-routing save
Routing:
- net GND: track 191.4 -> 641.8 mm, vias 56 -> 626
- net ROW3: track 383.0 -> 430.4 mm
- net ROW2: track 395.3 -> 434.2 mm
- net COL12: track 229.7 -> 240.9 mm
- net ROW5: track 516.4 -> 525.8 mm, vias 18 -> 20
- net VCC_LED_2: track 45.1 -> 52.0 mm
- net VCC_2: track 1258.6 -> 1265.4 mm, vias 36 -> 38
- net COL13: track 197.2 -> 203.9 mm
- net LED_PWR_EN: track 409.1 -> 415.3 mm, vias 15 -> 17
- net MOSI: track 429.8 -> 435.5 mm
- net LED15: track 226.7 -> 232.1 mm
- net RED10: track 217.3 -> 221.7 mm
- net LED13: track 231.6 -> 235.9 mm
- net BLU9: track 275.3 -> 271.1 mm
- net LED14: track 306.4 -> 310.4 mm
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Other:
- board text added: "99"
- board text added: "L O U I S E"
- board text added: "VR"

Commit message: Beta 1
Parts:
- removed Q0: 2N7002, ts_custom_nick_nacks:SOT23-3
- removed U_LED1, U_LED2: IS31FL3743B, ts_kb_mcu:UQFN40
- added Q3: 2N7002, ts_custom_nick_nacks:SOT23-3
- added U7, U8: TPS22995H-Q1, __untitled:SOT-23-THIN-6_DDC_TEX
- U5, U6: value TPS22995H-Q1 -> IS31FL3743B; device __untitled:SOT-23-THIN-6_DDC_TEX -> ts_kb_mcu:UQFN40
- moved Q1 233.2 mm to (305.7, 101.5), turned to 90 degrees
- moved U5 18.4 mm to (30.0, 58.0), turned to 45 degrees
- moved U6 17.9 mm to (248.5, 50.8), turned to 45 degrees
- moved Q2 16.5 mm to (88.5, 16.5)
- renumbered EEP to EEPROM, T2 to Q4, T3 to Q5
Connections:
- removed net N$10: JDIP.NC1, JDIP.NC2
- net GND: now also Q3.2, U5.16, U5.23, U5.EPAD, U5.EPAD@1, U5.EPAD@2, U6.16, U6.23, U6.EPAD, U6.EPAD@1, U6.EPAD@2, U7.4, U8.4; no longer Q0.2, U5.4, U6.4, U_LED1.16, U_LED1.23, U_LED1.EPAD, U_LED1.EPAD@1, U_LED1.EPAD@2, U_LED2.16, U_LED2.23, U_LED2.EPAD, U_LED2.EPAD@1, U_LED2.EPAD@2
- net LATCH: now also Q1.3; no longer Q0.3
- net LED1: now also U5.11; no longer U_LED1.11
- net LED10: now also U5.1; no longer U_LED1.1
- net LED11: now also U6.11; no longer U_LED2.11
- net LED12: now also U6.10; no longer U_LED2.10
- net LED13: now also U6.9; no longer U_LED2.9
- net LED14: now also U6.8; no longer U_LED2.8
- net LED15: now also U6.7; no longer U_LED2.7
- net LED16: now also U6.6; no longer U_LED2.6
- net LED17: now also U6.4; no longer U_LED2.4
- net LED18: now also U6.3; no longer U_LED2.3
- net LED19: now also U6.2; no longer U_LED2.2
- net LED1_CS: now also U5.25; no longer U_LED1.25
- net LED2: now also U5.10; no longer U_LED1.10
- net LED20: now also U6.1; no longer U_LED2.1
- net LED2_CS: now also U6.25; no longer U_LED2.25
- net LED3: now also U5.9; no longer U_LED1.9
- net LED4: now also U5.8; no longer U_LED1.8
- net LED5: now also U5.7; no longer U_LED1.7
- net LED6: now also U5.6; no longer U_LED1.6
- net LED7: now also U5.4; no longer U_LED1.4
- net LED8: now also U5.3; no longer U_LED1.3
- net LED9: now also U5.2; no longer U_LED1.2
- net LED_PWR_EN: now also U5.26, U6.26, U7.3, U8.3; no longer U5.3, U6.3, U_LED1.26, U_LED2.26
- net MATRIX_CS: now also Q1.1; no longer Q0.1
- net MISO: now also U5.24, U6.24; no longer U_LED1.24, U_LED2.24
- net MOSI: now also U5.28, U6.28; no longer U_LED1.28, U_LED2.28
- net N$1: now also U8.6; no longer U6.6
- net N$11: now also Q2.3; no longer Q1.3
- net N$12: now also Q2.1; no longer Q1.1
- net N$135: now also U7.6; no longer U5.6
- net N$136: now also U5.29; no longer U_LED1.29
- net N$151: now also U6.29; no longer U_LED2.29
- net N$7: now also Q3.3; no longer Q2.3
- net N$9: now also Q3.1; no longer Q2.1
- net SCK: now also U5.27, U6.27; no longer U_LED1.27, U_LED2.27
- net SYNC: now also U5.30, U6.30; no longer U_LED1.30, U_LED2.30
- net VCC_1: now also U7.1, U7.2, U8.1, U8.2; no longer U5.1, U5.2, U6.1, U6.2
- net VCC_LED_1: now also U5.22, U7.5; no longer U_LED1.22, U_LED1.5
- net VCC_LED_2: now also U6.22, U8.5; no longer U_LED2.22, U_LED2.5
- net XB1: now also U5.39; no longer U_LED1.39
- net XB10: now also U6.21; no longer U_LED2.21
- net XB11: now also U6.18; no longer U_LED2.18
- net XB12: now also U6.14; no longer U_LED2.14
- net XB2: now also U5.36; no longer U_LED1.36
- net XB3: now also U5.33; no longer U_LED1.33
- net XB4: now also U5.21; no longer U_LED1.21
- net XB5: now also U5.18; no longer U_LED1.18
- net XB6: now also U5.14; no longer U_LED1.14
- net XB7: now also U6.39; no longer U_LED2.39
- net XB8: now also U6.36; no longer U_LED2.36
- net XB9: now also U6.33; no longer U_LED2.33
- net XG1: now also U5.38; no longer U_LED1.38
- net XG10: now also U6.20; no longer U_LED2.20
- net XG11: now also U6.17; no longer U_LED2.17
- net XG12: now also U6.13; no longer U_LED2.13
- net XG2: now also U5.35; no longer U_LED1.35
- net XG3: now also U5.32; no longer U_LED1.32
- net XG4: now also U5.20; no longer U_LED1.20
- net XG5: now also U5.17; no longer U_LED1.17
- net XG6: now also U5.13; no longer U_LED1.13
- net XG7: now also U6.38; no longer U_LED2.38
- net XG8: now also U6.35; no longer U_LED2.35
- net XG9: now also U6.32; no longer U_LED2.32
- net XR1: now also U5.37; no longer U_LED1.37
- net XR10: now also U6.19; no longer U_LED2.19
- net XR11: now also U6.15; no longer U_LED2.15
- net XR12: now also U6.12; no longer U_LED2.12
- net XR2: now also U5.34; no longer U_LED1.34
- net XR3: now also U5.31; no longer U_LED1.31
- net XR4: now also U5.19; no longer U_LED1.19
- net XR5: now also U5.15; no longer U_LED1.15
- net XR6: now also U5.12; no longer U_LED1.12
- net XR7: now also U6.37; no longer U_LED2.37
- net XR8: now also U6.34; no longer U_LED2.34
- net XR9: now also U6.31; no longer U_LED2.31
Routing:
- net VCC_2: track 1265.4 -> 1319.4 mm, vias 38 -> 42
- net GND: track 641.8 -> 690.6 mm, vias 626 -> 655
- net ROW1: track 420.1 -> 462.2 mm
- net ROW4: track 446.3 -> 479.4 mm
- net COL2: track 179.3 -> 188.9 mm, vias 6 -> 7
- net ROW2: track 434.2 -> 443.2 mm
- net RED8: track 256.9 -> 261.2 mm
- net LED_PWR_EN: track 415.3 -> 411.0 mm, vias 17 -> 15
- net GRN9: track 319.1 -> 314.9 mm
- net J_RST: track 31.6 -> 34.9 mm
- net BLU11: track 230.4 -> 233.6 mm
- net N$92: track 5.15 -> 8.15 mm
- net N$44: track 5.15 -> 8.14 mm
- net N$49: track 5.15 -> 8.13 mm
- net N$99: track 5.15 -> 8.13 mm
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Other:
- board text added: "MG-M2"

Commit message: Added "ground to boot" function
Parts:
- added Q6: BSH201, ts_custom_nick_nacks:SOT23-3
- added R28, R29: 100K, rcl:R0603
- moved LOGO1 259.1 mm to (361.0, 46.0)
- moved C29 0.55 mm to (70.0, 19.9)
Connections:
- removed net N$13: D100.A, R26.2, RST.2, S1.3, S1.4
- new net !BOOT: Q6.1, R28.2, RST.2, S1.3, S1.4
- new net BOOT: D100.A, Q6.3, R26.2, R29.2
- net GND: now also R29.1, RST.1, S1.1, S1.2
- net VCC_2: now also Q6.2, R28.1; no longer RST.1, S1.1, S1.2
Routing:
- net N$13: track 38.2 -> 0.00 mm, vias 2 -> 0
- net BOOT: track 0.00 -> 35.4 mm, vias 0 -> 3
- net !BOOT: track 0.00 -> 25.9 mm, vias 0 -> 1
- net VCC_2: track 1319.4 -> 1297.8 mm, vias 42 -> 41
- net GND: track 690.6 -> 695.8 mm
- net XB4: track 18.6 -> 20.7 mm
- net LED5: track 243.9 -> 241.8 mm
- net VCC_LED_2: track 51.2 -> 52.3 mm
- net LED19: track 267.1 -> 266.4 mm
- net VCC_1: track 556.5 -> 557.2 mm
- net SDA: track 164.2 -> 164.8 mm
- net SCL: track 163.8 -> 164.4 mm
- net ROW5: track 528.4 -> 527.7 mm
- net N$11: track 19.2 -> 18.6 mm

Commit message: .
Parts:
- added C35, C36: 100nF, rcl:C0603
- added Q7: 2N7002, ts_custom_nick_nacks:SOT23-3
- added R30, R31: 5.1K, rcl:R0603
- added R32: 10K, rcl:R0603
- added R33@1: 0R, rcl:R0805W
- added R33@2, R34: 0R-DNP, rcl:R0805W
- added U$7: ??, tecsmith_jlcpcb_ordering:JLC_ORDER_NUMBER_QR_8X8
- EEPROM: value M25C -> M25CDUAL; device ts_kb_mcu:8-SOIC -> __tecsmith_kb_mcu:8-SOIC-SO8_N_W_DUAL
- moved D87 4.47 mm to (354.0, 18.0)
- moved C32 2.95 mm to (361.0, 98.7)
- moved R17 2.71 mm to (287.4, 113.4)
- moved R16 2.71 mm to (287.4, 111.3)
- moved U$5 2.70 mm to (174.6, 23.3)
- moved C31 1.64 mm to (361.0, 104.8)
- moved C28 0.65 mm to (284.4, 43.8)
Connections:
- removed net N$110: D91.A, SW_SPC.1@1, SW_SPC.1@2
- removed net PA8: JPWM.3, U1.29
- removed net PB5: JPWM.4, U1.41
- new net D91_A: D91.A, Q7.2, R34.2
- new net ENC_C: C31.1, R30.1, SW_F17.A, U1.29
- new net ENC_D: C32.1, R31.1, SW_F17.B, U1.41
- new net N$3: R33@1.2, R33@2.1, SW_SPC.2@1, SW_SPC.2@2
- net AUX_CS: now also JPWM.4
- net AUX_DC: now also JPWM.3
- net ENC_A: now also C35.1; no longer C31.1, SW_F17.A
- net ENC_B: now also C36.1; no longer C32.1, SW_F17.B
- net GND: now also C35.2, C36.2, R32.2
- net ROW5: now also Q7.3, R33@2.2; no longer SW_SPC.2@1, SW_SPC.2@2
- net VCC_2: now also R30.2, R31.2, R33@1.1
- net WKUP: now also Q7.1, R32.1, R34.1, SW_SPC.1@1, SW_SPC.1@2
Routing:
- net WKUP: track 62.1 -> 292.7 mm, vias 2 -> 12
- net ENC_C: track 0.00 -> 155.7 mm, vias 0 -> 7
- net ENC_D: track 0.00 -> 145.1 mm, vias 0 -> 7
- net ENC_A: track 198.0 -> 94.1 mm, vias 9 -> 6
- net ENC_B: track 199.8 -> 96.1 mm, vias 7 -> 5
- net PA8: track 87.8 -> 0.00 mm, vias 4 -> 0
- net PB5: track 84.9 -> 0.00 mm, vias 4 -> 0
- net VCC_2: track 1297.8 -> 1321.7 mm, vias 41 -> 43
- net AUX_CS: track 58.4 -> 80.5 mm, vias 2 -> 3
- net N$3: track 0.00 -> 14.3 mm, vias 0 -> 1
- net ROW5: track 527.7 -> 541.7 mm, vias 20 -> 24
- net AUX_DC: track 64.9 -> 76.1 mm, vias 3 -> 4
- net N$110: track 8.13 -> 0.00 mm
- net D91_A: track 0.00 -> 6.47 mm
- net GND: track 695.8 -> 701.3 mm, vias 655 -> 672
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Other:
- board text added: "PA1"
- board text added: "PB1"
- board text removed: "PA8"
- board text removed: "PB5"

Commit message: confirmed m2 mounting points
Parts:
- moved G6 1.50 mm to (22.3, 19.3)
- moved Z103 0.90 mm to (290.5, 77.3)
- moved Z102 0.37 mm to (290.5, 87.8)
- moved G2 0.34 mm to (201.3, 102.4)
- moved Z101 0.17 mm to (290.5, 98.7)
Routing:
- net GRN9: track 314.8 -> 317.1 mm
- net GND: track 701.3 -> 702.4 mm, vias 672 -> 674
- net COL1: track 226.7 -> 227.5 mm
- net LED14: track 309.9 -> 310.6 mm
- net COL12: track 240.7 -> 241.3 mm
- net BLU9: track 270.0 -> 269.5 mm
- net RED6: track 348.7 -> 348.4 mm, vias 11 -> 12
- net ROW5: track 541.7 -> 541.9 mm, vias 24 -> 22
Other:
- outline, holes or cut-outs redrawn

Commit message: .
Parts:
- added TP-3V3, TP-5V, TP-GND, TP-LED-EN, TP-USB+, TP-USB-, TP-V-LED-1, TP-V-LED-2: TEST-POINT.3SQ, tecsmith_keyboards:PAD.03X.03-SQ
Connections:
- net GND: now also TP-GND.1
- net LED_PWR_EN: now also TP-LED-EN.1
- net USB_D_N: now also TP-USB-.1
- net USB_D_P: now also TP-USB+.1
- net VCC_1: now also TP-5V.1
- net VCC_2: now also TP-3V3.1
- net VCC_LED_1: now also TP-V-LED-1.1
- net VCC_LED_2: now also TP-V-LED-2.1
Routing:
- net VCC_2: track 1321.7 -> 1326.8 mm
- net GND: track 702.4 -> 699.4 mm
- net VCC_1: track 557.2 -> 559.3 mm
- net USB_D_N: track 289.7 -> 291.8 mm
- net USB_D_P: track 291.7 -> 293.7 mm
- net LED_PWR_EN: track 411.8 -> 412.5 mm
- net VCC_LED_1: track 77.1 -> 77.6 mm
Other:
- board text added: "5V"
- board text added: "D+"
- board text added: "D-"
