File: EAGLE/vr99/vr99-revA.sch (EAGLE design)
At the start: 455 parts, among them Q1 2N7002, Q2 2N7002, Q3 2N7002, Q4 AO3401A, Q5 AO3401A, Q6 BSH201, Q7 2N7002, U1 STM32F411CEU7THERM, U2 74HC589A_DT, U3 74HC589A_DT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

Commit message: .
Parts:
- added TP-3V3, TP-5V, TP-GND, TP-LED-EN, TP-USB+, TP-USB-, TP-V-LED-1, TP-V-LED-2: TEST-POINT.3SQ, tecsmith_keyboards:TEST-POINT.3SQ
Connections:
- net GND: now also TP-GND.1
- net LED_PWR_EN: now also TP-LED-EN.1
- net USB_D_N: now also TP-USB-.1
- net USB_D_P: now also TP-USB+.1
- net VCC_1: now also TP-5V.1
- net VCC_2: now also TP-3V3.1
- net VCC_LED_1: now also TP-V-LED-1.1
- net VCC_LED_2: now also TP-V-LED-2.1
Changed lines of the file:
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@@
 <part name="R33@1" library="rcl" library_urn="urn:adsk.eagle:library:334" deviceset="R-EU_" device="R0805W" package3d_urn="urn:adsk.eagle:package:23537/2" value="0R"/>
 <part name="U$7" library="tecsmith_jlcpcb_ordering" deviceset="JLC_ORDER_NUMBER_QR" device="QR_8X8" value="??"/>
+<part name="TP-5V" library="tecsmith_keyboards" deviceset="TEST-POINT" device=".3SQ"/>
+<part name="TP-3V3" library="tecsmith_keyboards" deviceset="TEST-POINT" device=".3SQ"/>
+<part name="TP-USB+" library="tecsmith_keyboards" deviceset="TEST-POINT" device=".3SQ"/>
+<part name="TP-USB-" library="tecsmith_keyboards" deviceset="TEST-POINT" device=".3SQ"/>
+<part name="TP-LED-EN" library="tecsmith_keyboards" deviceset="TEST-POINT" device=".3SQ"/>
+<part name="TP-V-LED-1" library="tecsmith_keyboards" deviceset="TEST-POINT" device=".3SQ"/>
+<part name="TP-V-LED-2" library="tecsmith_keyboards" deviceset="TEST-POINT" device=".3SQ"/>
+<part name="TP-GND" library="tecsmith_keyboards" deviceset="TEST-POINT" device=".3SQ"/>
 </parts>
 <sheets>
@@
 <attribute name="VALUE" x="54.61" y="40.64" size="1.778" layer="96" font="vector" align="top-left"/>
 </instance>
+<instance part="TP-5V" gate="G$1" x="10.16" y="27.94" smashed="yes">
+<attribute name="NAME" x="11.938" y="27.178" size="1.27" layer="104"/>
+</instance>
+<instance part="TP-3V3" gate="G$1" x="45.72" y="27.94" smashed="yes">
+<attribute name="NAME" x="47.498" y="27.432" size="1.27" layer="104"/>
+</instance>
+<instance part="TP-USB+" gate="G$1" x="210.82" y="58.42" smashed="yes">
+<attribute name="NAME" x="209.042" y="58.928" size="1.27" layer="104" rot="R180"/>
+</instance>
+<instance part="TP-USB-" gate="G$1" x="218.44" y="58.42" smashed="yes">
+<attribute name="NAME" x="220.218" y="57.912" size="1.27" layer="104"/>
+</instance>
+<instance part="TP-GND" gate="G$1" x="45.72" y="7.62" smashed="yes">
+<attribute name="NAME" x="47.498" y="7.112" size="1.27" layer="104"/>
+</instance>
 </instances>
 <busses>
@@
 <pinref part="D00" gate="G$1" pin="A"/>
 <wire x1="38.1" y1="25.4" x2="40.64" y2="25.4" width="0.1524" layer="91"/>
-<wire x1="40.64" y1="25.4" x2="50.8" y2="25.4" width="0.1524" layer="91"/>
+<wire x1="40.64" y1="25.4" x2="45.72" y2="25.4" width="0.1524" layer="91"/>
+<wire x1="45.72" y1="25.4" x2="50.8" y2="25.4" width="0.1524" layer="91"/>
 <wire x1="30.48" y1="33.02" x2="38.1" y2="33.02" width="0.1524" layer="91"/>
 <wire x1="38.1" y1="33.02" x2="38.1" y2="25.4" width="0.1524" layer="91"/>
@@
 <wire x1="40.64" y1="22.86" x2="40.64" y2="25.4" width="0.1524" layer="91"/>
 <junction x="40.64" y="25.4"/>
+<pinref part="TP-3V3" gate="G$1" pin="1"/>
+<wire x1="45.72" y1="27.94" x2="45.72" y2="25.4" width="0.1524" layer="91"/>
+<junction x="45.72" y="25.4"/>
 </segment>
 <segment>
@@
 <wire x1="15.24" y1="10.16" x2="27.94" y2="10.16" width="0.1524" layer="91"/>
 <pinref part="C22" gate="G$1" pin="2"/>
-<wire x1="27.94" y1="10.16" x2="50.8" y2="10.16" width="0.1524" layer="91"/>
+<wire x1="27.94" y1="10.16" x2="45.72" y2="10.16" width="0.1524" layer="91"/>
+<wire x1="45.72" y1="10.16" x2="50.8" y2="10.16" width="0.1524" layer="91"/>
 <wire x1="50.8" y1="10.16" x2="50.8" y2="12.7" width="0.1524" layer="91"/>
 <junction x="27.94" y="10.16"/>
@@
 <wire x1="73.66" y1="10.16" x2="71.12" y2="10.16" width="0.1524" layer="91"/>
 <junction x="71.12" y="10.16"/>
+<pinref part="TP-GND" gate="G$1" pin="1"/>
+<wire x1="45.72" y1="10.16" x2="45.72" y2="7.62" width="0.1524" layer="91"/>
+<junction x="45.72" y="10.16"/>
 </segment>
 <segment>
@@
 </segment>
 <segment>
-<wire x1="215.9" y1="48.26" x2="215.9" y2="55.88" width="0.1524" layer="91"/>
-<label x="215.9" y="55.88" size="1.27" layer="95" rot="R90" xref="yes"/>
+<wire x1="215.9" y1="48.26" x2="215.9" y2="58.42" width="0.1524" layer="91"/>
+<label x="215.9" y="60.96" size="1.27" layer="95" rot="R90" xref="yes"/>
 <pinref part="UDB1" gate="J1" pin="DN"/>
+<pinref part="TP-USB-" gate="G$1" pin="1"/>
+<wire x1="215.9" y1="58.42" x2="215.9" y2="60.96" width="0.1524" layer="91"/>
+<wire x1="218.44" y1="58.42" x2="215.9" y2="58.42" width="0.1524" layer="91"/>
+<junction x="215.9" y="58.42"/>
 </segment>
 <segment>
@@
 <net name="VCC_1" class="0">
 <segment>
-<wire x1="15.24" y1="25.4" x2="5.08" y2="25.4" width="0.1524" layer="91"/>
+<wire x1="15.24" y1="25.4" x2="10.16" y2="25.4" width="0.1524" layer="91"/>
 <junction x="15.24" y="25.4"/>
 <pinref part="C21" gate="G$1" pin="1"/>
+<wire x1="10.16" y1="25.4" x2="5.08" y2="25.4" width="0.1524" layer="91"/>
 <wire x1="15.24" y1="20.32" x2="15.24" y2="25.4" width="0.1524" layer="91"/>
 <pinref part="C20" gate="G$1" pin="1"/>
@@
 <wire x1="5.08" y1="30.48" x2="5.08" y2="25.4" width="0.1524" layer="91"/>
 <junction x="5.08" y="25.4"/>
+<pinref part="TP-5V" gate="G$1" pin="1"/>
+<wire x1="10.16" y1="27.94" x2="10.16" y2="25.4" width="0.1524" layer="91"/>
+<junction x="10.16" y="25.4"/>
 </segment>
 <segment>
@@
 </segment>
 <segment>
-<wire x1="213.36" y1="48.26" x2="213.36" y2="55.88" width="0.1524" layer="91"/>
-<label x="213.36" y="55.88" size="1.27" layer="95" rot="R90" xref="yes"/>
+<wire x1="213.36" y1="48.26" x2="213.36" y2="58.42" width="0.1524" layer="91"/>
+<label x="213.36" y="60.96" size="1.27" layer="95" rot="R90" xref="yes"/>
 <pinref part="UDB1" gate="J1" pin="DP"/>
+<pinref part="TP-USB+" gate="G$1" pin="1"/>
+<wire x1="213.36" y1="58.42" x2="213.36" y2="60.96" width="0.1524" layer="91"/>
+<wire x1="210.82" y1="58.42" x2="213.36" y2="58.42" width="0.1524" layer="91"/>
+<junction x="213.36" y="58.42"/>
 </segment>
 <segment>
@@
 <attribute name="VALUE" x="355.092" y="16.51" size="2.54" layer="96"/>
 </instance>
+<instance part="TP-LED-EN" gate="G$1" x="327.66" y="58.42" smashed="yes">
+<attribute name="NAME" x="329.438" y="57.912" size="1.27" layer="104"/>
+</instance>
+<instance part="TP-V-LED-1" gate="G$1" x="355.6" y="76.2" smashed="yes">
+<attribute name="NAME" x="357.378" y="75.692" size="1.27" layer="104"/>
+</instance>
+<instance part="TP-V-LED-2" gate="G$1" x="355.6" y="48.26" smashed="yes">
+<attribute name="NAME" x="357.378" y="47.752" size="1.27" layer="104"/>
+</instance>
 </instances>
 <busses>
@@
 <wire x1="325.12" y1="58.42" x2="325.12" y2="66.04" width="0.1524" layer="91"/>
 <wire x1="325.12" y1="66.04" x2="327.66" y2="66.04" width="0.1524" layer="91"/>
+<pinref part="TP-LED-EN" gate="G$1" pin="1"/>
+<wire x1="325.12" y1="58.42" x2="327.66" y2="58.42" width="0.1524" layer="91"/>
+<junction x="325.12" y="58.42"/>
 </segment>
 <segment>
@@
 <wire x1="355.6" y1="71.12" x2="355.6" y2="73.66" width="0.1524" layer="91"/>
 <wire x1="355.6" y1="73.66" x2="360.68" y2="73.66" width="0.1524" layer="91"/>
+<pinref part="TP-V-LED-1" gate="G$1" pin="1"/>
+<wire x1="355.6" y1="76.2" x2="355.6" y2="73.66" width="0.1524" layer="91"/>
+<junction x="355.6" y="73.66"/>
 </segment>
 </net>
@@
 <wire x1="355.6" y1="43.18" x2="355.6" y2="45.72" width="0.1524" layer="91"/>
 <wire x1="355.6" y1="45.72" x2="360.68" y2="45.72" width="0.1524" layer="91"/>
+<pinref part="TP-V-LED-2" gate="G$1" pin="1"/>
+<wire x1="355.6" y1="48.26" x2="355.6" y2="45.72" width="0.1524" layer="91"/>
+<junction x="355.6" y="45.72"/>
 </segment>
 </net>
