File: KiCAD/sr99-stm32f411-hotswap/sr99-stm32f411-hotswap-common-mcu.kicad_sch (KiCad schematic)
At the start: 1 part, among them U1 STM32F411C_C-E_Ux

Commit message: wip-2025-11-17
Parts:
- added C1, C2, C3, C5, C6: 100n, Capacitor_SMD:C_0603_1608Metric, symbol ts-kicad-lib:C
- added C4, C7: 22u, Capacitor_SMD:C_0603_1608Metric, symbol ts-kicad-lib:C
- added C8: 4u7, Capacitor_SMD:C_0603_1608Metric, symbol ts-kicad-lib:C
- added D1: 1N4148WS, Diode_SMD:D_SOD-323_HandSoldering, symbol ts-kicad-lib:D
- added Q1: 2N7002, Package_TO_SOT_SMD:SOT-23, symbol Transistor_FET:2N7002
- added R1, R2, R3, R4, R5: 10K, Resistor_SMD:R_Array_Convex_4x0603, symbol ts-kicad-lib:R_Array04
- added R6: 10K, Capacitor_SMD:C_0603_1608Metric, symbol ts-kicad-lib:R
- added R7: 5K1, Capacitor_SMD:C_0603_1608Metric, symbol ts-kicad-lib:R
- added U2, U3, U4: MC74HC589AD, Package_SO:TSSOP-16_4.4x5mm_P0.65mm, symbol ts-kicad-lib:MC74HC589AD
- added U5: AMS1117-3.3, Package_TO_SOT_SMD:SOT-223-3_TabPin2, symbol Regulator_Linear:AMS1117-3.3
Connections:
- new net: R6.2, U4.1 (B), U4.15 (A), U4.2 (C), U4.3 (D)
- new net: U3.9 (QH), U4.14 (SA)
- new net: R4.2, U2.15 (A)
- new net: U2.9 (QH), U3.14 (SA)
- new net: R5.2, U3.15 (A)
- new net +3V3: C1.2, C2.2, C3.2, C6.2, C7.2, C8.2, D1.2 (A), R7.1, U2.16 (VCC), U3.16 (VCC), U4.16 (VCC), U5.2 (VO)
- new net +5V: C4.2, C5.2, D1.1 (K), U5.3 (VI)
- new net COL0: R4.4, U2.1 (B)
- new net COL1: R4.6, U2.2 (C)
- new net COL10: R2.2, U3.4 (E)
- new net COL11: R2.4, U3.5 (F)
- new net COL12: R2.6, U3.6 (G)
- new net COL13: R2.8, U3.7 (H)
- new net COL14: R3.2, U4.4 (E)
- new net COL15: R3.4, U4.5 (F)
- new net COL16: R3.6, U4.6 (G)
- new net COL17: R3.8, U4.7 (H)
- new net COL2: R4.8, U2.3 (D)
- new net COL3: R1.2, U2.4 (E)
- new net COL4: R1.4, U2.5 (F)
- new net COL5: R1.6, U2.6 (G)
- new net COL6: R1.8, U2.7 (H)
- new net COL7: R5.4, U3.1 (B)
- new net COL8: R5.6, U3.2 (C)
- new net COL9: R5.8, U3.3 (D)
- new net GND: C1.1, C2.1, C3.1, C4.1, C5.1, C6.1, C7.1, C8.1, Q1.2 (S), R1.1, R1.3, R1.5, R1.7, R2.1, R2.3, R2.5, R2.7, R3.1, R3.3, R3.5, R3.7, R4.1, R4.3, R4.5, R4.7, R5.1, R5.3, R5.5, R5.7, R6.1, U2.14 (SA), U2.8 (GND), U3.8 (GND), U4.8 (GND), U5.1 (GND)
- new net LATCH: Q1.3 (D), R7.2, U2.12 (LATCH), U2.13 (SS/*PL), U3.12 (LATCH), U3.13 (SS/*PL), U4.12 (LATCH), U4.13 (SS/*PL)
- new net MATRIX_CS: Q1.1 (G), U2.10 (OE/CS), U3.10 (OE/CS), U4.10 (OE/CS)
- new net MISO: U4.9 (QH)
- new net SCK: U2.11 (SC/SCK), U3.11 (SC/SCK), U4.11 (SC/SCK)
Other:
- note added: "Column Scanner"
- note added: "Power Supply"
- moved on the sheet: U1
