File: KiCAD/sr99-stm32f411-hotswap/sr99-stm32f411-hotswap-matrix.kicad_sch (KiCad schematic)
At the start: 224 parts, among them Q1 AO3401A, Q2 AO3401A, SW1 Esc, SW10 F9, SW100_1 Menu, SW101 Fn1, SW102_1 Fn2, SW103 Left, SW104 Down, SW105 Right, SW106 N0, SW107 Dot, SW11 F10, SW12 F11, SW13 F12, SW14 F13, SW15 F14, SW16 F15, SW17 F16, SW18 F17, SW2 F1, SW20 1, SW21 2, SW22 3, SW23 4, SW24 5, SW25 6, SW26 7, SW27 8, SW28 9, SW29 0, SW3 F2, SW30 MIN, SW31 PLS, SW32 BS, SW33 NumL, SW34 Div, SW35 Mul, SW36 Sub, SW37 Tab, SW38 Q, SW39 W, SW4 F3, SW40 E, SW41 R, SW42 T, SW43 Y, SW44 U, SW45 I, SW46 O, SW47 P, SW48 [, SW49 ], SW5 F4, SW50 \, SW51 N7, SW52 N8, SW53 N9, SW54 Add, SW55 CapsL, SW56 A, SW57 S, SW58 D, SW59 F, SW6 F5, SW60 G, SW61 H, SW62 J, SW63 K, SW64 L, SW65 ;, SW66 ", SW68 Ent, SW69 N4, SW7 F6, SW70 N5, SW71 N6, SW73 LShft, SW75 Z, SW76 X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

Commit message: wip-2025-11-17
Parts:
- removed D1, D19: 1N4148WS, Diode_SMD:D_SOD-323_HandSoldering, symbol ts-kicad-lib:D_45deg
- removed R4, R8: 10K, Resistor_SMD:R_0603_1608Metric_Pad0.98x0.95mm_HandSolder, symbol Device:R_Small
- removed R5, R6, R7, R9: 5.1K, Resistor_SMD:R_0603_1608Metric_Pad0.98x0.95mm_HandSolder, symbol Device:R_Small
- added D20, D4: 1N4148WS, Diode_SMD:D_SOD-323_HandSoldering, symbol ts-kicad-lib:D_45deg
- added R8, R9: 10K, symbol ts-kicad-lib:R_Array04
- SW19: value ~ -> Tdl
- renumbered C4 to C10, C5 to C11, C6 to C12, C3 to C9, D9 to D10, D102 to D100, D103 to D101, D104 to D102, D105 to D103, D106 to D104, D107 to D105, D10 to D11, D11 to D12, D12 to D13, D13 to D14, D14 to D15, D15 to D16, D16 to D17, D17 to D18, D18 to D19, D20 to D21, D21 to D22, D22 to D23, D23 to D24, D24 to D25, D25 to D26, D26 to D27, D27 to D28, D28 to D29, D29 to D30, D30 to D31, D31 to D32, D32 to D33, D33 to D34, D34 to D35, D35 to D36, D36 to D37, D37 to D38, D38 to D39, D39 to D40, D40 to D41, D41 to D42, D42 to D43, D43 to D44, D44 to D45, D45 to D46, D46 to D47, D47 to D48, D48 to D49, D4 to D5, D49 to D50, D50 to D51, D51 to D52, D52 to D53, D53 to D54, D54 to D55, D94 to D56, D95 to D57, D96 to D58, D98 to D59, D5 to D6, D99 to D60, D55 to D61, D56 to D62, D57 to D63, D58 to D64, D59 to D65, D60 to D66, D61 to D67, D62 to D68, D63 to D69, D6 to D7, D64 to D70, D65 to D71, D66 to D72, D68 to D73, D69 to D74, D70 to D75, D71 to D76, D73 to D77, D75 to D78, D76 to D79, D7 to D8, D77 to D80, D78 to D81, D79 to D82, D80 to D83, D81 to D84, D82 to D85, D83 to D86, D84 to D87, D85 to D88, D86 to D89, D8 to D9, D87 to D90, D88 to D91, D89 to D92, D90 to D93, D91 to D94, D92 to D95, D93 to D96, D100 to D98, D101 to D99, Q1 to Q2, Q2 to Q3, ST5 to ST2, ST2 to ST3, ST3 to ST4, ST6 to ST5, ST4 to ST6, SW68 to SW67, SW69 to SW68, SW70 to SW69, SW71 to SW70, SW73 to SW71, SW75 to SW72, SW76 to SW73, SW77 to SW74, SW78 to SW75, SW79 to SW76, SW80 to SW77, SW81 to SW78, SW82 to SW79, SW83 to SW80, SW84 to SW81, SW85 to SW82, SW86 to SW83, SW87 to SW84, SW88 to SW85, SW89 to SW86, SW90 to SW87, SW91 to SW88, SW92 to SW89, SW93 to SW90, SW97 to SW91, SW101 to SW92, SW103 to SW93, SW104 to SW94, SW94-5-6-8-9 to SW94-5-6-8-1, SW105 to SW95, SW106 to SW96, SW107 to SW97
Connections:
- net +3V3: now also R8.2, R8.4, R8.8, R9.2, R9.4, R9.8
- net COL0: now also D2.1 (K), D20.1 (K)
- net COL1: now also D3.1 (K); no longer D2.1 (K)
- net COL2: now also D4.1 (K); no longer D3.1 (K)
- net ENC_A: now also R8.1
- net ENC_B: now also R8.3
- net ENC_C: now also R9.1, R9.3
- net GND: now also ENC1.G, ENC2.G; no longer ENC1.C, ENC2.C
- net at Q2.1 (G): now also ENC1.E, R8.7; no longer ENC1.S
- net at Q3.1 (G): now also ENC2.E, R9.7; no longer ENC2.S
- net at SW3.1: now also D4.2 (A); no longer D3.2 (A)
- net at SW1.1: now also D2.2 (A)
- net at SW2.1: now also D3.2 (A); no longer D2.2 (A)
- net at SW19.1: now also D20.2 (A)
- no-connect marks 0 -> 4
Other:
- moved on the sheet: Q2, Q3
