File: KiCAD/sr99-stm32f411-hotswap/sr99-stm32f411-hotswap.kicad_sch (KiCad schematic)
At the start: 0 parts

Commit message: wip-2025-11-17
Other:
- sheet ARGB renamed ARGB Driver
- added sheet ARGB Matrix (sr99-stm32f411-hotswap-argb2.kicad_sch)
- sheet ARGB Driver: file sr99-stm32f411-hotswap-argb.kicad_sch -> sr99-stm32f411-hotswap-argb1.kicad_sch
- note added: "ARGB Driver ↓"
- note added: "ARGB Matrix ↓"
- note removed: "ARGB ↓"
Changed lines of the file:
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@@
 	(generator_version "9.0")
 	(paper "A4")
-	(text "ARGB\n↓"
+	(text "ARGB Driver\n↓"
 		(exclude_from_sim no)
-		(at 238.252 87.63 0)
+		(at 178.308 103.124 0)
 		(effects
 			(font
@@
 	(text "MCU\n↓"
 		(exclude_from_sim no)
-		(at 57.15 87.376 0)
+		(at 54.102 102.87 0)
+		(effects
+			(font
+				(size 3.81 3.81)
+				(thickness 0.4763)
+			)
+		)
+	)
+	(text "ARGB Matrix\n↓"
+		(exclude_from_sim no)
+		(at 240.03 103.378 0)
 		(effects
 			(font
@@
 	(text "Matrix\n↓"
 		(exclude_from_sim no)
-		(at 148.336 87.376 0)
+		(at 115.824 102.87 0)
 		(effects
 			(font
@@
 	(image
 		(at 145.7869 62.5345)
-		(scale 0.209293)
+		(scale 0.352791)
 		(data "iVBORw0KGgoAAAANSUhEUgAAEMwAAAXSCAMAAADN7jRHAAABsFBMVEUAAAD7+/vu7u7S0tLMzMyq"
 			"qqr9/f0AAAC8vLyZmZm3t7fKysq1tbWpqam4uLjPz88DAwPd3d0ICAjs7OyJiYkGBgaYmJje3t4K"
@@
 	)
 	(sheet
-		(at 109.22 93.98)
-		(size 76.2 50.8)
+		(at 210.82 109.22)
+		(size 59.69 36.83)
+		(exclude_from_sim no)
+		(in_bom yes)
+		(on_board yes)
+		(dnp no)
+		(fields_autoplaced yes)
+		(stroke
+			(width 0.1524)
+			(type solid)
+		)
+		(fill
+			(color 0 0 0 0.0000)
+		)
+		(property "Sheetname" "ARGB Matrix"
+			(at 210.82 108.5084 0)
+			(effects
+				(font
+					(size 1.27 1.27)
+				)
+				(justify left bottom)
+			)
+		)
+		(property "Sheetfile" "sr99-stm32f411-hotswap-argb2.kicad_sch"
+			(at 210.82 146.6346 0)
+			(effects
+				(font
+					(size 1.27 1.27)
+				)
+				(justify left top)
+			)
+		)
+		(instances
+			(project "sr99-stm32f411-hotswap"
+				(path "/e21675ae-fe46-4cba-befb-5225609570c3"
+					(page "5")
+				)
+			)
+		)
+	)
+	(sheet
+		(at 86.36 109.22)
+		(size 59.69 36.83)
 		(exclude_from_sim no)
 		(in_bom yes)
@@
 		)
 		(property "Sheetname" "Matrix"
-			(at 109.22 93.2684 0)
+			(at 86.36 108.5084 0)
 			(effects
 				(font
@@
 		)
 		(property "Sheetfile" "sr99-stm32f411-hotswap-matrix.kicad_sch"
-			(at 109.22 145.3646 0)
+			(at 86.36 146.6346 0)
 			(effects
 				(font
@@
 	)
 	(sheet
-		(at 20.32 93.98)
-		(size 76.2 50.8)
+		(at 24.13 109.22)
+		(size 59.69 36.83)
 		(exclude_from_sim no)
 		(in_bom yes)
@@
 		)
 		(property "Sheetname" "MCU and power"
-			(at 20.32 93.2684 0)
+			(at 24.13 108.5084 0)
 			(effects
 				(font
@@
 		)
 		(property "Sheetfile" "sr99-stm32f411-hotswap-common-mcu.kicad_sch"
-			(at 20.32 145.3646 0)
+			(at 24.13 146.6346 0)
 			(effects
 				(font
@@
 	)
 	(sheet
-		(at 198.12 93.98)
-		(size 76.2 50.8)
+		(at 148.59 109.22)
+		(size 59.69 36.83)
 		(exclude_from_sim no)
 		(in_bom yes)
@@
 			(color 0 0 0 0.0000)
 		)
-		(property "Sheetname" "ARGB"
-			(at 198.12 93.2684 0)
+		(property "Sheetname" "ARGB Driver"
+			(at 148.59 108.5084 0)
 			(effects
 				(font
@@
 			)
 		)
-		(property "Sheetfile" "sr99-stm32f411-hotswap-argb.kicad_sch"
-			(at 198.12 145.3646 0)
+		(property "Sheetfile" "sr99-stm32f411-hotswap-argb1.kicad_sch"
+			(at 148.59 146.6346 0)
 			(effects
 				(font
