File: KiCAD/sr99-stm32-hotswap/sr99-stm32-hotswap-argb2.kicad_sch (KiCad schematic)
At the start: 106 parts

Commit message: update-2025-11-20
Parts:
- W35, W36: footprint ts-keyboard-lib:RGB-156120M -> ts-keyboard-lib:RGB-156120M_VIA
Changed lines of the file:
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@@
 			)
 		)
-		(property "Footprint" "ts-keyboard-lib:RGB-156120M"
+		(property "Footprint" "ts-keyboard-lib:RGB-156120M_VIA"
 			(at 354.33 94.234 0)
 			(effects
@@
 			)
 		)
-		(property "Footprint" "ts-keyboard-lib:RGB-156120M"
+		(property "Footprint" "ts-keyboard-lib:RGB-156120M_VIA"
 			(at 372.11 94.234 0)
 			(effects

Commit message: wip
Parts:
- W1, W10, W100, W101, W102, W103, W104, W105, W106, W11, W12, W13, W14, W15, W16, W17, W18, W19, W2, W20, W21, W22, W23, W24, W25, W26, W27, W28, W29, W3, W30, W31, W32, W33, W34, W37, W38, W39, W4, W40, W41, W42, W43, W44, W45, W46, W47, W48, W49, W5, W50, W51, W52, W53, W54, W55, W56, W57, W58, W59, W6, W60, W61, W62, W63, W64, W65, W66, W67, W68, W69, W7, W70, W71, W72, W73, W74, W75, W76, W77, W78, W79, W8, W80, W81, W82, W83, W84, W85, W86, W87, W88, W89, W9, W90, W91, W92, W93, W94, W95, W96, W97, W98, W99: footprint ts-keyboard-lib:RGB-156120M -> ts-keyboard-lib:RGB-3528; symbol ts-keyboard-lib:RGB_Comm_Anode -> ts-keyboard-lib:Comm_Anode_RGB4
- W35, W36: footprint ts-keyboard-lib:RGB-156120M_VIA -> ts-keyboard-lib:RGB-3528; symbol ts-keyboard-lib:RGB_Comm_Anode -> ts-keyboard-lib:Comm_Anode_RGB4
Connections:
- net BLU1: now also W1.3 (B), W2.3 (B), W3.3 (B), W4.3 (B), W5.3 (B), W6.3 (B), W7.3 (B), W8.3 (B), W9.3 (B); no longer W1.2 (B), W2.2 (B), W3.2 (B), W4.2 (B), W5.2 (B), W6.2 (B), W7.2 (B), W8.2 (B), W9.2 (B)
- net BLU10: now also W63.3 (B), W64.3 (B), W65.3 (B), W66.3 (B), W67.3 (B), W68.3 (B), W69.3 (B), W70.3 (B); no longer W63.2 (B), W64.2 (B), W65.2 (B), W66.2 (B), W67.2 (B), W68.2 (B), W69.2 (B), W70.2 (B)
- net BLU11: now also W79.3 (B), W80.3 (B), W81.3 (B), W82.3 (B), W83.3 (B), W84.3 (B), W85.3 (B), W86.3 (B); no longer W79.2 (B), W80.2 (B), W81.2 (B), W82.2 (B), W83.2 (B), W84.2 (B), W85.2 (B), W86.2 (B)
- net BLU12: now also W100.3 (B), W101.3 (B), W102.3 (B), W103.3 (B), W95.3 (B), W96.3 (B), W97.3 (B), W98.3 (B), W99.3 (B); no longer W100.2 (B), W101.2 (B), W102.2 (B), W103.2 (B), W95.2 (B), W96.2 (B), W97.2 (B), W98.2 (B), W99.2 (B)
- net BLU2: now also W19.3 (B), W20.3 (B), W21.3 (B), W22.3 (B), W23.3 (B), W24.3 (B), W25.3 (B), W26.3 (B), W27.3 (B); no longer W19.2 (B), W20.2 (B), W21.2 (B), W22.2 (B), W23.2 (B), W24.2 (B), W25.2 (B), W26.2 (B), W27.2 (B)
- net BLU3: now also W104.3 (B), W37.3 (B), W38.3 (B), W39.3 (B), W40.3 (B), W41.3 (B), W42.3 (B), W43.3 (B), W44.3 (B), W45.3 (B); no longer W104.2 (B), W37.2 (B), W38.2 (B), W39.2 (B), W40.2 (B), W41.2 (B), W42.2 (B), W43.2 (B), W44.2 (B), W45.2 (B)
- net BLU4: now also W105.3 (B), W54.3 (B), W55.3 (B), W56.3 (B), W57.3 (B), W58.3 (B), W59.3 (B), W60.3 (B), W61.3 (B), W62.3 (B); no longer W105.2 (B), W54.2 (B), W55.2 (B), W56.2 (B), W57.2 (B), W58.2 (B), W59.2 (B), W60.2 (B), W61.2 (B), W62.2 (B)
- net BLU5: now also W106.3 (B), W71.3 (B), W72.3 (B), W73.3 (B), W74.3 (B), W75.3 (B), W76.3 (B), W77.3 (B), W78.3 (B); no longer W106.2 (B), W71.2 (B), W72.2 (B), W73.2 (B), W74.2 (B), W75.2 (B), W76.2 (B), W77.2 (B), W78.2 (B)
- net BLU6: now also W87.3 (B), W88.3 (B), W89.3 (B), W90.3 (B), W91.3 (B), W92.3 (B), W93.3 (B), W94.3 (B); no longer W87.2 (B), W88.2 (B), W89.2 (B), W90.2 (B), W91.2 (B), W92.2 (B), W93.2 (B), W94.2 (B)
- net BLU7: now also W10.3 (B), W11.3 (B), W12.3 (B), W13.3 (B), W14.3 (B), W15.3 (B), W16.3 (B), W17.3 (B), W18.3 (B); no longer W10.2 (B), W11.2 (B), W12.2 (B), W13.2 (B), W14.2 (B), W15.2 (B), W16.2 (B), W17.2 (B), W18.2 (B)
- net BLU8: now also W28.3 (B), W29.3 (B), W30.3 (B), W31.3 (B), W32.3 (B), W33.3 (B), W34.3 (B), W35.3 (B), W36.3 (B); no longer W28.2 (B), W29.2 (B), W30.2 (B), W31.2 (B), W32.2 (B), W33.2 (B), W34.2 (B), W35.2 (B), W36.2 (B)
- net BLU9: now also W46.3 (B), W47.3 (B), W48.3 (B), W49.3 (B), W50.3 (B), W51.3 (B), W52.3 (B), W53.3 (B); no longer W46.2 (B), W47.2 (B), W48.2 (B), W49.2 (B), W50.2 (B), W51.2 (B), W52.2 (B), W53.2 (B)
- net GRN1: now also W1.2 (G), W2.2 (G), W3.2 (G), W4.2 (G), W5.2 (G), W6.2 (G), W7.2 (G), W8.2 (G), W9.2 (G); no longer W1.4 (G), W2.4 (G), W3.4 (G), W4.4 (G), W5.4 (G), W6.4 (G), W7.4 (G), W8.4 (G), W9.4 (G)
- net GRN10: now also W63.2 (G), W64.2 (G), W65.2 (G), W66.2 (G), W67.2 (G), W68.2 (G), W69.2 (G), W70.2 (G); no longer W63.4 (G), W64.4 (G), W65.4 (G), W66.4 (G), W67.4 (G), W68.4 (G), W69.4 (G), W70.4 (G)
- net GRN11: now also W79.2 (G), W80.2 (G), W81.2 (G), W82.2 (G), W83.2 (G), W84.2 (G), W85.2 (G), W86.2 (G); no longer W79.4 (G), W80.4 (G), W81.4 (G), W82.4 (G), W83.4 (G), W84.4 (G), W85.4 (G), W86.4 (G)
- net GRN12: now also W100.2 (G), W101.2 (G), W102.2 (G), W103.2 (G), W95.2 (G), W96.2 (G), W97.2 (G), W98.2 (G), W99.2 (G); no longer W100.4 (G), W101.4 (G), W102.4 (G), W103.4 (G), W95.4 (G), W96.4 (G), W97.4 (G), W98.4 (G), W99.4 (G)
- net GRN2: now also W19.2 (G), W20.2 (G), W21.2 (G), W22.2 (G), W23.2 (G), W24.2 (G), W25.2 (G), W26.2 (G), W27.2 (G); no longer W19.4 (G), W20.4 (G), W21.4 (G), W22.4 (G), W23.4 (G), W24.4 (G), W25.4 (G), W26.4 (G), W27.4 (G)
- net GRN3: now also W104.2 (G), W37.2 (G), W38.2 (G), W39.2 (G), W40.2 (G), W41.2 (G), W42.2 (G), W43.2 (G), W44.2 (G), W45.2 (G); no longer W104.4 (G), W37.4 (G), W38.4 (G), W39.4 (G), W40.4 (G), W41.4 (G), W42.4 (G), W43.4 (G), W44.4 (G), W45.4 (G)
- net GRN4: now also W105.2 (G), W54.2 (G), W55.2 (G), W56.2 (G), W57.2 (G), W58.2 (G), W59.2 (G), W60.2 (G), W61.2 (G), W62.2 (G); no longer W105.4 (G), W54.4 (G), W55.4 (G), W56.4 (G), W57.4 (G), W58.4 (G), W59.4 (G), W60.4 (G), W61.4 (G), W62.4 (G)
- net GRN5: now also W106.2 (G), W71.2 (G), W72.2 (G), W73.2 (G), W74.2 (G), W75.2 (G), W76.2 (G), W77.2 (G), W78.2 (G); no longer W106.4 (G), W71.4 (G), W72.4 (G), W73.4 (G), W74.4 (G), W75.4 (G), W76.4 (G), W77.4 (G), W78.4 (G)
- net GRN6: now also W87.2 (G), W88.2 (G), W89.2 (G), W90.2 (G), W91.2 (G), W92.2 (G), W93.2 (G), W94.2 (G); no longer W87.4 (G), W88.4 (G), W89.4 (G), W90.4 (G), W91.4 (G), W92.4 (G), W93.4 (G), W94.4 (G)
- net GRN7: now also W10.2 (G), W11.2 (G), W12.2 (G), W13.2 (G), W14.2 (G), W15.2 (G), W16.2 (G), W17.2 (G), W18.2 (G); no longer W10.4 (G), W11.4 (G), W12.4 (G), W13.4 (G), W14.4 (G), W15.4 (G), W16.4 (G), W17.4 (G), W18.4 (G)
- net GRN8: now also W28.2 (G), W29.2 (G), W30.2 (G), W31.2 (G), W32.2 (G), W33.2 (G), W34.2 (G), W35.2 (G), W36.2 (G); no longer W28.4 (G), W29.4 (G), W30.4 (G), W31.4 (G), W32.4 (G), W33.4 (G), W34.4 (G), W35.4 (G), W36.4 (G)
- net GRN9: now also W46.2 (G), W47.2 (G), W48.2 (G), W49.2 (G), W50.2 (G), W51.2 (G), W52.2 (G), W53.2 (G); no longer W46.4 (G), W47.4 (G), W48.4 (G), W49.4 (G), W50.4 (G), W51.4 (G), W52.4 (G), W53.4 (G)
- net LED1: now also W1.4 (+), W19.4 (+), W37.4 (+), W54.4 (+), W71.4 (+), W87.4 (+); no longer W1.1 (+), W19.1 (+), W37.1 (+), W54.1 (+), W71.1 (+), W87.1 (+)
- net LED10: now also W104.4 (+), W105.4 (+), W106.4 (+); no longer W104.1 (+), W105.1 (+), W106.1 (+)
- net LED11: now also W10.4 (+), W28.4 (+), W46.4 (+), W63.4 (+), W79.4 (+), W95.4 (+); no longer W10.1 (+), W28.1 (+), W46.1 (+), W63.1 (+), W79.1 (+), W95.1 (+)
- net LED12: now also W11.4 (+), W29.4 (+), W47.4 (+), W64.4 (+), W80.4 (+), W96.4 (+); no longer W11.1 (+), W29.1 (+), W47.1 (+), W64.1 (+), W80.1 (+), W96.1 (+)
- net LED13: now also W12.4 (+), W30.4 (+), W48.4 (+), W65.4 (+), W81.4 (+), W97.4 (+); no longer W12.1 (+), W30.1 (+), W48.1 (+), W65.1 (+), W81.1 (+), W97.1 (+)
- net LED14: now also W13.4 (+), W31.4 (+), W49.4 (+), W82.4 (+), W98.4 (+); no longer W13.1 (+), W31.1 (+), W49.1 (+), W82.1 (+), W98.1 (+)
- net LED15: now also W14.4 (+), W32.4 (+), W50.4 (+), W66.4 (+), W83.4 (+), W99.4 (+); no longer W14.1 (+), W32.1 (+), W50.1 (+), W66.1 (+), W83.1 (+), W99.1 (+)
- net LED16: now also W100.4 (+), W15.4 (+), W33.4 (+), W67.4 (+), W84.4 (+); no longer W100.1 (+), W15.1 (+), W33.1 (+), W67.1 (+), W84.1 (+)
- net LED17: now also W101.4 (+), W16.4 (+), W34.4 (+), W51.4 (+), W68.4 (+), W85.4 (+); no longer W101.1 (+), W16.1 (+), W34.1 (+), W51.1 (+), W68.1 (+), W85.1 (+)
- net LED18: now also W102.4 (+), W17.4 (+), W35.4 (+), W52.4 (+), W69.4 (+), W86.4 (+); no longer W102.1 (+), W17.1 (+), W35.1 (+), W52.1 (+), W69.1 (+), W86.1 (+)
- net LED19: now also W103.4 (+), W18.4 (+), W36.4 (+), W53.4 (+), W70.4 (+); no longer W103.1 (+), W18.1 (+), W36.1 (+), W53.1 (+), W70.1 (+)
- net LED2: now also W2.4 (+), W20.4 (+), W38.4 (+), W55.4 (+), W88.4 (+); no longer W2.1 (+), W20.1 (+), W38.1 (+), W55.1 (+), W88.1 (+)
- net LED3: now also W21.4 (+), W3.4 (+), W39.4 (+), W56.4 (+), W72.4 (+), W89.4 (+); no longer W21.1 (+), W3.1 (+), W39.1 (+), W56.1 (+), W72.1 (+), W89.1 (+)
- net LED4: now also W22.4 (+), W4.4 (+), W40.4 (+), W57.4 (+), W73.4 (+); no longer W22.1 (+), W4.1 (+), W40.1 (+), W57.1 (+), W73.1 (+)
- net LED5: now also W23.4 (+), W41.4 (+), W5.4 (+), W58.4 (+), W74.4 (+), W90.4 (+); no longer W23.1 (+), W41.1 (+), W5.1 (+), W58.1 (+), W74.1 (+), W90.1 (+)
- net LED6: now also W24.4 (+), W42.4 (+), W59.4 (+), W6.4 (+), W75.4 (+), W91.4 (+); no longer W24.1 (+), W42.1 (+), W59.1 (+), W6.1 (+), W75.1 (+), W91.1 (+)
- net LED7: now also W25.4 (+), W43.4 (+), W60.4 (+), W7.4 (+), W76.4 (+), W92.4 (+); no longer W25.1 (+), W43.1 (+), W60.1 (+), W7.1 (+), W76.1 (+), W92.1 (+)
- net LED8: now also W26.4 (+), W44.4 (+), W61.4 (+), W77.4 (+), W8.4 (+), W93.4 (+); no longer W26.1 (+), W44.1 (+), W61.1 (+), W77.1 (+), W8.1 (+), W93.1 (+)
- net LED9: now also W27.4 (+), W45.4 (+), W62.4 (+), W78.4 (+), W9.4 (+), W94.4 (+); no longer W27.1 (+), W45.1 (+), W62.1 (+), W78.1 (+), W9.1 (+), W94.1 (+)
- net RED1: now also W1.1 (R), W2.1 (R), W3.1 (R), W4.1 (R), W5.1 (R), W6.1 (R), W7.1 (R), W8.1 (R), W9.1 (R); no longer W1.3 (R), W2.3 (R), W3.3 (R), W4.3 (R), W5.3 (R), W6.3 (R), W7.3 (R), W8.3 (R), W9.3 (R)
- net RED10: now also W63.1 (R), W64.1 (R), W65.1 (R), W66.1 (R), W67.1 (R), W68.1 (R), W69.1 (R), W70.1 (R); no longer W63.3 (R), W64.3 (R), W65.3 (R), W66.3 (R), W67.3 (R), W68.3 (R), W69.3 (R), W70.3 (R)
- net RED11: now also W79.1 (R), W80.1 (R), W81.1 (R), W82.1 (R), W83.1 (R), W84.1 (R), W85.1 (R), W86.1 (R); no longer W79.3 (R), W80.3 (R), W81.3 (R), W82.3 (R), W83.3 (R), W84.3 (R), W85.3 (R), W86.3 (R)
- net RED12: now also W100.1 (R), W101.1 (R), W102.1 (R), W103.1 (R), W95.1 (R), W96.1 (R), W97.1 (R), W98.1 (R), W99.1 (R); no longer W100.3 (R), W101.3 (R), W102.3 (R), W103.3 (R), W95.3 (R), W96.3 (R), W97.3 (R), W98.3 (R), W99.3 (R)
- net RED2: now also W19.1 (R), W20.1 (R), W21.1 (R), W22.1 (R), W23.1 (R), W24.1 (R), W25.1 (R), W26.1 (R), W27.1 (R); no longer W19.3 (R), W20.3 (R), W21.3 (R), W22.3 (R), W23.3 (R), W24.3 (R), W25.3 (R), W26.3 (R), W27.3 (R)
- net RED3: now also W104.1 (R), W37.1 (R), W38.1 (R), W39.1 (R), W40.1 (R), W41.1 (R), W42.1 (R), W43.1 (R), W44.1 (R), W45.1 (R); no longer W104.3 (R), W37.3 (R), W38.3 (R), W39.3 (R), W40.3 (R), W41.3 (R), W42.3 (R), W43.3 (R), W44.3 (R), W45.3 (R)
- net RED4: now also W105.1 (R), W54.1 (R), W55.1 (R), W56.1 (R), W57.1 (R), W58.1 (R), W59.1 (R), W60.1 (R), W61.1 (R), W62.1 (R); no longer W105.3 (R), W54.3 (R), W55.3 (R), W56.3 (R), W57.3 (R), W58.3 (R), W59.3 (R), W60.3 (R), W61.3 (R), W62.3 (R)
- net RED5: now also W106.1 (R), W71.1 (R), W72.1 (R), W73.1 (R), W74.1 (R), W75.1 (R), W76.1 (R), W77.1 (R), W78.1 (R); no longer W106.3 (R), W71.3 (R), W72.3 (R), W73.3 (R), W74.3 (R), W75.3 (R), W76.3 (R), W77.3 (R), W78.3 (R)
- net RED6: now also W87.1 (R), W88.1 (R), W89.1 (R), W90.1 (R), W91.1 (R), W92.1 (R), W93.1 (R), W94.1 (R); no longer W87.3 (R), W88.3 (R), W89.3 (R), W90.3 (R), W91.3 (R), W92.3 (R), W93.3 (R), W94.3 (R)
- net RED7: now also W10.1 (R), W11.1 (R), W12.1 (R), W13.1 (R), W14.1 (R), W15.1 (R), W16.1 (R), W17.1 (R), W18.1 (R); no longer W10.3 (R), W11.3 (R), W12.3 (R), W13.3 (R), W14.3 (R), W15.3 (R), W16.3 (R), W17.3 (R), W18.3 (R)
- net RED8: now also W28.1 (R), W29.1 (R), W30.1 (R), W31.1 (R), W32.1 (R), W33.1 (R), W34.1 (R), W35.1 (R), W36.1 (R); no longer W28.3 (R), W29.3 (R), W30.3 (R), W31.3 (R), W32.3 (R), W33.3 (R), W34.3 (R), W35.3 (R), W36.3 (R)
- net RED9: now also W46.1 (R), W47.1 (R), W48.1 (R), W49.1 (R), W50.1 (R), W51.1 (R), W52.1 (R), W53.1 (R); no longer W46.3 (R), W47.3 (R), W48.3 (R), W49.3 (R), W50.3 (R), W51.3 (R), W52.3 (R), W53.3 (R)
Other:
- moved on the sheet: W100, W101, W102, W103, W104, W105, W106, W19, W20, W21, W22, W23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

Commit message: pre-DRC upload
Connections:
- net BLU10: now also W106.3 (B)
- net BLU3: no longer W104.3 (B)
- net BLU4: no longer W105.3 (B)
- net BLU5: no longer W106.3 (B)
- net BLU8: now also W104.3 (B)
- net BLU9: now also W105.3 (B)
- net GRN10: now also W106.2 (G)
- net GRN3: no longer W104.2 (G)
- net GRN4: no longer W105.2 (G)
- net GRN5: no longer W106.2 (G)
- net GRN8: now also W104.2 (G)
- net GRN9: now also W105.2 (G)
- net RED10: now also W106.1 (R)
- net RED3: no longer W104.1 (R)
- net RED4: no longer W105.1 (R)
- net RED5: no longer W106.1 (R)
- net RED8: now also W104.1 (R)
- net RED9: now also W105.1 (R)
